File: PCB/16-STEPPER-DRIVER-CARD/16-STEPPER-DRIVER-CARD.kicad_sch (KiCad schematic)
At the start: 33 parts

Commit message: PCB Routing for Stepper Card
Parts:
- removed A10, A11, A12, A13, A14, A15, A16, A9: Pololu_Breakout_A4988, Module:Pololu_Breakout-16_15.2x20.3mm, symbol Driver_Motor:Pololu_Breakout_A4988
- removed C10, C11, C12, C13, C14, C15, C16, C9: C_Polarized_US, symbol Device:C_Polarized_US
- A1, A2, A3, A4, A5, A6, A7, A8: value Pololu_Breakout_A4988 -> (none)
- C1, C2, C3, C4, C5, C6, C7, C8: value C_Polarized_US -> (none)
- gave numbers to parts that had none: 1
Connections:
- net +5V: now also J1.59, J1.60
- net A1EN: now also J1.15
- net A1MS1: now also J1.17
- net A1MS2: now also J1.19; no longer A6.11 (MS2)
- net A1MS3: now also J1.21
- net A1STEP: now also J1.13
- net A2EN: now also J1.27
- net A2MS1: now also J1.29
- net A2MS2: now also J1.31
- net A2MS3: now also J1.33
- net A2STEP: now also J1.25
- net A3EN: now also J1.39
- net A3MS1: now also J1.41
- net A3MS2: now also J1.43
- net A3MS3: now also J1.45
- net A3STEP: now also J1.37
- net A4EN: now also J1.51
- net A4MS1: now also J1.53
- net A4MS2: now also J1.55
- net A4MS3: now also J1.57
- net A4STEP: now also J1.49
- net A5EN: now also J1.16
- net A5MS1: now also J1.18
- net A5MS2: now also J1.20
- net A5MS3: now also J1.22
- net A5STEP: now also J1.14
- net A6EN: now also J1.28
- net A6MS1: now also J1.30
- net A6MS3: now also J1.34
- net A6STEP: now also J1.26
- net A7EN: now also J1.40
- net A7MS1: now also J1.42
- net A7MS2: now also J1.44
- net A7MS3: now also J1.46
- net A7STEP: now also J1.38
- net A8EN: now also J1.52
- net A8MS1: now also J1.54
- net A8MS2: now also J1.56
- net A8MS3: now also J1.58
- net A8STEP: now also J1.50
- net DIR1: now also J1.11; no longer A2.16 (DIR)
- net DIR2: now also A2.16 (DIR), J1.23; no longer A3.16 (DIR), A4.16 (DIR)
- net DIR3: now also A3.16 (DIR), J1.35; no longer A5.16 (DIR), A6.16 (DIR)
- net DIR4: now also A4.16 (DIR), J1.47; no longer A7.16 (DIR), A8.16 (DIR)
- net GND: now also J1.01, J1.02, J1.03, J1.04
- net VCC: now also J1.05, J1.06, J1.07, J1.08, J1.09, J1.10
- net DIR5: now reaches J1.12
- net DIR5: now also A5.16 (DIR)
- net DIR6: now reaches J1.24
- net DIR6: now also A6.16 (DIR)
- net A6MS2: now reaches J1.32
- net A6MS2: now also A6.11 (MS2)
- net DIR7: now reaches J1.36
- net DIR7: now also A7.16 (DIR)
- net DIR8: now reaches J1.48
- net DIR8: now also A8.16 (DIR)
- no-connect marks 64 -> 32
Other:
- moved on the sheet: A1, A2, A3, A4, A5, A6, A7, A8, C1, C2, C3, C4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

Commit message: ignore
Parts:
- A1, A2, A3, A4, A5, A6, A7, A8: value (none) -> Pololu_Breakout_A4988
- C1, C2, C3, C4, C5, C6, C7, C8: value (none) -> C_Polarized_US; footprint (none) -> Capacitor_THT:CP_Radial_D6.3mm_P2.50mm
- J1: value (none) -> MEC2-30-01-X-TH1-NP-WT; footprint (none) -> LIBRARIES:MEC2-30-01-J-TH1-NP-WT-EDGECARD
Changed lines of the file:
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@@
       (effects (font (size 1.27 1.27)) (justify left))
     )
-    (property "Value" "" (id 1) (at 191.77 241.3 0)
-      (effects (font (size 1.27 1.27)) (justify left))
-    )
-    (property "Footprint" "" (id 2) (at 199.39 233.68 0)
+    (property "Value" "C_Polarized_US" (id 1) (at 191.77 241.3 0)
+      (effects (font (size 1.27 1.27)) (justify left))
+    )
+    (property "Footprint" "Capacitor_THT:CP_Radial_D6.3mm_P2.50mm" (id 2) (at 199.39 233.68 0)
       (effects (font (size 1.27 1.27)) hide)
     )
@@
       (effects (font (size 1.27 1.27)) (justify left))
     )
-    (property "Value" "" (id 1) (at 116.3194 89.0071 0)
+    (property "Value" "Pololu_Breakout_A4988" (id 1) (at 116.3194 89.0071 0)
       (effects (font (size 1.27 1.27)) (justify left))
     )
@@
       (effects (font (size 1.27 1.27)) (justify left))
     )
-    (property "Value" "" (id 1) (at 140.97 238.76 0)
-      (effects (font (size 1.27 1.27)) (justify left))
-    )
-    (property "Footprint" "" (id 2) (at 148.59 233.68 0)
+    (property "Value" "C_Polarized_US" (id 1) (at 140.97 238.76 0)
+      (effects (font (size 1.27 1.27)) (justify left))
+    )
+    (property "Footprint" "Capacitor_THT:CP_Radial_D6.3mm_P2.50mm" (id 2) (at 148.59 233.68 0)
       (effects (font (size 1.27 1.27)) hide)
     )
@@
       (effects (font (size 1.27 1.27)) hide)
     )
-    (property "Value" "" (id 1) (at 219.71 194.31 0))
+    (property "Value" "+5V" (id 1) (at 219.71 194.31 0))
     (property "Footprint" "" (id 2) (at 219.71 189.23 0)
       (effects (font (size 1.27 1.27)) hide)
@@
       (effects (font (size 1.27 1.27)) (justify left))
     )
-    (property "Value" "" (id 1) (at 161.29 238.76 0)
-      (effects (font (size 1.27 1.27)) (justify left))
-    )
-    (property "Footprint" "" (id 2) (at 168.91 233.68 0)
+    (property "Value" "C_Polarized_US" (id 1) (at 161.29 238.76 0)
+      (effects (font (size 1.27 1.27)) (justify left))
+    )
+    (property "Footprint" "Capacitor_THT:CP_Radial_D6.3mm_P2.50mm" (id 2) (at 168.91 233.68 0)
       (effects (font (size 1.27 1.27)) hide)
     )
@@
       (effects (font (size 1.27 1.27)) hide)
     )
-    (property "Value" "" (id 1) (at 140.97 196.2134 0))
+    (property "Value" "GND" (id 1) (at 140.97 196.2134 0))
     (property "Footprint" "" (id 2) (at 140.97 191.77 0)
       (effects (font (size 1.27 1.27)) hide)
@@
       (effects (font (size 1.27 1.27)) (justify left))
     )
-    (property "Value" "" (id 1) (at 261.0994 29.3171 0)
+    (property "Value" "Pololu_Breakout_A4988" (id 1) (at 261.0994 29.3171 0)
       (effects (font (size 1.27 1.27)) (justify left))
     )
@@
       (effects (font (size 1.27 1.27)) (justify left))
     )
-    (property "Value" "" (id 1) (at 210.2994 29.3171 0)
+    (property "Value" "Pololu_Breakout_A4988" (id 1) (at 210.2994 29.3171 0)
       (effects (font (size 1.27 1.27)) (justify left))
     )
@@
       (effects (font (size 1.27 1.27)) (justify left))
     )
-    (property "Value" "" (id 1) (at 151.13 241.3 0)
-      (effects (font (size 1.27 1.27)) (justify left))
-    )
-    (property "Footprint" "" (id 2) (at 158.75 233.68 0)
+    (property "Value" "C_Polarized_US" (id 1) (at 151.13 241.3 0)
+      (effects (font (size 1.27 1.27)) (justify left))
+    )
+    (property "Footprint" "Capacitor_THT:CP_Radial_D6.3mm_P2.50mm" (id 2) (at 158.75 233.68 0)
       (effects (font (size 1.27 1.27)) hide)
     )
@@
       (effects (font (size 1.27 1.27)) (justify left))
     )
-    (property "Value" "" (id 1) (at 130.81 241.3 0)
-      (effects (font (size 1.27 1.27)) (justify left))
-    )
-    (property "Footprint" "" (id 2) (at 138.43 233.68 0)
+    (property "Value" "C_Polarized_US" (id 1) (at 130.81 241.3 0)
+      (effects (font (size 1.27 1.27)) (justify left))
+    )
+    (property "Footprint" "Capacitor_THT:CP_Radial_D6.3mm_P2.50mm" (id 2) (at 138.43 233.68 0)
       (effects (font (size 1.27 1.27)) hide)
     )
@@
       (effects (font (size 1.27 1.27)) (justify left))
     )
-    (property "Value" "" (id 1) (at 266.1794 89.0071 0)
+    (property "Value" "Pololu_Breakout_A4988" (id 1) (at 266.1794 89.0071 0)
       (effects (font (size 1.27 1.27)) (justify left))
     )
@@
       (effects (font (size 1.27 1.27)) (justify left))
     )
-    (property "Value" "" (id 1) (at 181.61 238.76 0)
-      (effects (font (size 1.27 1.27)) (justify left))
-    )
-    (property "Footprint" "" (id 2) (at 189.23 233.68 0)
+    (property "Value" "C_Polarized_US" (id 1) (at 181.61 238.76 0)
+      (effects (font (size 1.27 1.27)) (justify left))
+    )
+    (property "Footprint" "Capacitor_THT:CP_Radial_D6.3mm_P2.50mm" (id 2) (at 189.23 233.68 0)
       (effects (font (size 1.27 1.27)) hide)
     )
@@
       (effects (font (size 1.27 1.27)) (justify left))
     )
-    (property "Value" "" (id 1) (at 171.45 241.3 0)
-      (effects (font (size 1.27 1.27)) (justify left))
-    )
-    (property "Footprint" "" (id 2) (at 179.07 233.68 0)
+    (property "Value" "C_Polarized_US" (id 1) (at 171.45 241.3 0)
+      (effects (font (size 1.27 1.27)) (justify left))
+    )
+    (property "Footprint" "Capacitor_THT:CP_Radial_D6.3mm_P2.50mm" (id 2) (at 179.07 233.68 0)
       (effects (font (size 1.27 1.27)) hide)
     )
@@
       (effects (font (size 1.27 1.27)) (justify left))
     )
-    (property "Value" "" (id 1) (at 162.0394 29.3171 0)
+    (property "Value" "Pololu_Breakout_A4988" (id 1) (at 162.0394 29.3171 0)
       (effects (font (size 1.27 1.27)) (justify left))
     )
@@
       (effects (font (size 1.27 1.27)) (justify left))
     )
-    (property "Value" "" (id 1) (at 142.748 178.2322 90)
-      (effects (font (size 1.27 1.27)) (justify left))
-    )
-    (property "Footprint" "" (id 2) (at 181.61 176.53 0)
+    (property "Value" "MEC2-30-01-X-TH1-NP-WT" (id 1) (at 142.748 178.2322 90)
+      (effects (font (size 1.27 1.27)) (justify left))
+    )
+    (property "Footprint" "LIBRARIES:MEC2-30-01-J-TH1-NP-WT-EDGECARD" (id 2) (at 181.61 176.53 0)
       (effects (font (size 1.27 1.27)) (justify left bottom) hide)
     )
@@
       (effects (font (size 1.27 1.27)) (justify left))
     )
-    (property "Value" "" (id 1) (at 164.5794 89.0071 0)
+    (property "Value" "Pololu_Breakout_A4988" (id 1) (at 164.5794 89.0071 0)
       (effects (font (size 1.27 1.27)) (justify left))
     )
@@
       (effects (font (size 1.27 1.27)) (justify left))
     )
-    (property "Value" "" (id 1) (at 215.3794 89.0071 0)
+    (property "Value" "Pololu_Breakout_A4988" (id 1) (at 215.3794 89.0071 0)
       (effects (font (size 1.27 1.27)) (justify left))
     )
@@
       (effects (font (size 1.27 1.27)) (justify left))
     )
-    (property "Value" "" (id 1) (at 120.65 238.76 0)
-      (effects (font (size 1.27 1.27)) (justify left))
-    )
-    (property "Footprint" "" (id 2) (at 128.27 233.68 0)
+    (property "Value" "C_Polarized_US" (id 1) (at 120.65 238.76 0)
+      (effects (font (size 1.27 1.27)) (justify left))
+    )
+    (property "Footprint" "Capacitor_THT:CP_Radial_D6.3mm_P2.50mm" (id 2) (at 128.27 233.68 0)
       (effects (font (size 1.27 1.27)) hide)
     )
@@
       (effects (font (size 1.27 1.27)) (justify left))
     )
-    (property "Value" "" (id 1) (at 116.3194 29.3171 0)
-      (effects (font (size 1.27 1.27)) (justify left))
-    )
+    (property "Value" "Pololu_Breakout_A4988" (id 1) (at 116.3194 29.3171 0)
+      (effects (font (size 1.27 1.27)) (justify left))
+    )
