File: PCB/16-STEPPER-DRIVER-CARD/16-STEPPER-DRIVER-CARD.kicad_pcb (KiCad board)
At the start: 2 copper layers, 99.1 x 73 mm, 17 parts, among them J1 MEC2-30-01-X-TH1-NP-WT

Commit message: final rev 1 design, no slots
Other:
- outline, holes or cut-outs redrawn
- board text added: "8-STEPPER-DRIVER-CARD REV A ELLIOT EICKHOLTZ"
