File: PCB/16-STEPPER-DRIVER-CARD/8-STEPPER-DRIVER-CARD.kicad_pcb (KiCad board)
At the start: 2 copper layers, 99.1 x 73 mm, 17 parts, among them J1 MEC2-30-01-X-TH1-NP-WT

Commit message: Name change, final addition before prototype order
Parts:
- added J2: Conn_01x04_Male, Connector_PinHeader_2.54mm:PinHeader_1x04_P2.54mm_Vertical, F.Cu at (112.0, 58.2)
- added J3: Conn_01x04_Male, Connector_PinHeader_2.54mm:PinHeader_1x04_P2.54mm_Vertical, F.Cu at (136.7, 58.2)
- added J4: Conn_01x04_Male, Connector_PinHeader_2.54mm:PinHeader_1x04_P2.54mm_Vertical, F.Cu at (161.3, 58.2)
- added J5: Conn_01x04_Male, Connector_PinHeader_2.54mm:PinHeader_1x04_P2.54mm_Vertical, F.Cu at (185.9, 58.2)
- added J6: Conn_01x04_Male, Connector_PinHeader_2.54mm:PinHeader_1x04_P2.54mm_Vertical, F.Cu at (112.0, 86.6)
- added J7: Conn_01x04_Male, Connector_PinHeader_2.54mm:PinHeader_1x04_P2.54mm_Vertical, F.Cu at (136.7, 86.6)
- added J8: Conn_01x04_Male, Connector_PinHeader_2.54mm:PinHeader_1x04_P2.54mm_Vertical, F.Cu at (161.3, 86.6)
- added J9: Conn_01x04_Male, Connector_PinHeader_2.54mm:PinHeader_1x04_P2.54mm_Vertical, F.Cu at (185.9, 86.6)
Connections:
- A1 pad 3: unconnected-(A1-Pad3) -> Net-(A1-Pad3)
- A1 pad 4: unconnected-(A1-Pad4) -> Net-(A1-Pad4)
- A1 pad 5: unconnected-(A1-Pad5) -> Net-(A1-Pad5)
- A1 pad 6: unconnected-(A1-Pad6) -> Net-(A1-Pad6)
- A2 pad 3: unconnected-(A2-Pad3) -> Net-(A2-Pad3)
- A2 pad 4: unconnected-(A2-Pad4) -> Net-(A2-Pad4)
- A2 pad 5: unconnected-(A2-Pad5) -> Net-(A2-Pad5)
- A2 pad 6: unconnected-(A2-Pad6) -> Net-(A2-Pad6)
- A3 pad 3: unconnected-(A3-Pad3) -> Net-(A3-Pad3)
- A3 pad 4: unconnected-(A3-Pad4) -> Net-(A3-Pad4)
- A3 pad 5: unconnected-(A3-Pad5) -> Net-(A3-Pad5)
- A3 pad 6: unconnected-(A3-Pad6) -> Net-(A3-Pad6)
- A4 pad 3: unconnected-(A4-Pad3) -> Net-(A4-Pad3)
- A4 pad 4: unconnected-(A4-Pad4) -> Net-(A4-Pad4)
- A4 pad 5: unconnected-(A4-Pad5) -> Net-(A4-Pad5)
- A4 pad 6: unconnected-(A4-Pad6) -> Net-(A4-Pad6)
- A5 pad 3: unconnected-(A5-Pad3) -> Net-(A5-Pad3)
- A5 pad 4: unconnected-(A5-Pad4) -> Net-(A5-Pad4)
- A5 pad 5: unconnected-(A5-Pad5) -> Net-(A5-Pad5)
- A5 pad 6: unconnected-(A5-Pad6) -> Net-(A5-Pad6)
- A6 pad 3: unconnected-(A6-Pad3) -> Net-(A6-Pad3)
- A6 pad 4: unconnected-(A6-Pad4) -> Net-(A6-Pad4)
- A6 pad 5: unconnected-(A6-Pad5) -> Net-(A6-Pad5)
- A6 pad 6: unconnected-(A6-Pad6) -> Net-(A6-Pad6)
- A7 pad 3: unconnected-(A7-Pad3) -> Net-(A7-Pad3)
- A7 pad 4: unconnected-(A7-Pad4) -> Net-(A7-Pad4)
- A7 pad 5: unconnected-(A7-Pad5) -> Net-(A7-Pad5)
- A7 pad 6: unconnected-(A7-Pad6) -> Net-(A7-Pad6)
- A8 pad 3: unconnected-(A8-Pad3) -> Net-(A8-Pad3)
- A8 pad 4: unconnected-(A8-Pad4) -> Net-(A8-Pad4)
- A8 pad 5: unconnected-(A8-Pad5) -> Net-(A8-Pad5)
- A8 pad 6: unconnected-(A8-Pad6) -> Net-(A8-Pad6)
Routing:
- net Net-(A8-Pad6): track 0.00 -> 4.79 mm
- net Net-(A8-Pad5): track 0.00 -> 4.79 mm
- net Net-(A8-Pad4): track 0.00 -> 4.79 mm
- net Net-(A8-Pad3): track 0.00 -> 4.79 mm
- net Net-(A7-Pad6): track 0.00 -> 4.77 mm
- net Net-(A7-Pad5): track 0.00 -> 4.77 mm
- net Net-(A7-Pad4): track 0.00 -> 4.77 mm
- net Net-(A7-Pad3): track 0.00 -> 4.77 mm
- net Net-(A6-Pad6): track 0.00 -> 4.74 mm
- net Net-(A6-Pad5): track 0.00 -> 4.74 mm
- net Net-(A6-Pad4): track 0.00 -> 4.74 mm
- net Net-(A6-Pad3): track 0.00 -> 4.74 mm
- net Net-(A5-Pad6): track 0.00 -> 4.71 mm
- net Net-(A5-Pad5): track 0.00 -> 4.71 mm
- net Net-(A5-Pad4): track 0.00 -> 4.71 mm
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