File: PCB/16-STEPPER-DRIVER-CARD/8-STEPPER-DRIVER-CARD.kicad_sch (KiCad schematic)
At the start: 17 parts, among them J1 MEC2-30-01-X-TH1-NP-WT

Commit message: Name change, final addition before prototype order
Parts:
- added J2: (no value), symbol Connector:Conn_01x04_Male
- added J3, J4, J5, J6, J7, J8, J9: Conn_01x04_Male, symbol Connector:Conn_01x04_Male
Connections:
- net at A5.3 (1B): now also J6.1 (Pin_1)
- net at A5.4 (1A): now also J6.2 (Pin_2)
- net at A5.5 (2A): now also J6.3 (Pin_3)
- net at A5.6 (2B): now also J6.4 (Pin_4)
- net at A4.3 (1B): now also J5.1 (Pin_1)
- net at A4.4 (1A): now also J5.2 (Pin_2)
- net at A4.5 (2A): now also J5.3 (Pin_3)
- net at A4.6 (2B): now also J5.4 (Pin_4)
- net at A3.3 (1B): now also J4.1 (Pin_1)
- net at A3.4 (1A): now also J4.2 (Pin_2)
- net at A3.5 (2A): now also J4.3 (Pin_3)
- net at A3.6 (2B): now also J4.4 (Pin_4)
- net at A8.3 (1B): now also J9.1 (Pin_1)
- net at A8.4 (1A): now also J9.2 (Pin_2)
- net at A8.5 (2A): now also J9.3 (Pin_3)
- net at A8.6 (2B): now also J9.4 (Pin_4)
- net at A2.3 (1B): now also J3.1 (Pin_1)
- net at A2.4 (1A): now also J3.2 (Pin_2)
- net at A2.5 (2A): now also J3.3 (Pin_3)
- net at A2.6 (2B): now also J3.4 (Pin_4)
- net at A6.3 (1B): now also J7.1 (Pin_1)
- net at A6.4 (1A): now also J7.2 (Pin_2)
- net at A6.5 (2A): now also J7.3 (Pin_3)
- net at A6.6 (2B): now also J7.4 (Pin_4)
- net at A7.3 (1B): now also J8.1 (Pin_1)
- net at A7.4 (1A): now also J8.2 (Pin_2)
- net at A7.5 (2A): now also J8.3 (Pin_3)
- net at A7.6 (2B): now also J8.4 (Pin_4)
- net at A1.3 (1B): now also J2.1 (Pin_1)
- net at A1.4 (1A): now also J2.2 (Pin_2)
- net at A1.5 (2A): now also J2.3 (Pin_3)
- net at A1.6 (2B): now also J2.4 (Pin_4)
- no-connect marks 32 -> 0
Changed lines of the file:
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@@
   (junction (at 168.91 227.965) (diameter 0) (color 0 0 0 0)
   )
-  (no_connect (at 266.7 50.8))
-  (no_connect (at 167.64 48.26))
-  (no_connect (at 266.7 43.18))
-  (no_connect (at 266.7 48.26))
-  (no_connect (at 271.78 110.49))
-  (no_connect (at 215.9 43.18))
-  (no_connect (at 220.98 105.41))
-  (no_connect (at 215.9 48.26))
-  (no_connect (at 121.92 110.49))
-  (no_connect (at 215.9 45.72))
-  (no_connect (at 266.7 45.72))
-  (no_connect (at 170.18 105.41))
-  (no_connect (at 170.18 110.49))
-  (no_connect (at 271.78 105.41))
-  (no_connect (at 271.78 102.87))
-  (no_connect (at 167.64 50.8))
-  (no_connect (at 170.18 107.95))
-  (no_connect (at 220.98 102.87))
-  (no_connect (at 220.98 110.49))
-  (no_connect (at 167.64 45.72))
-  (no_connect (at 167.64 43.18))
-  (no_connect (at 121.92 102.87))
-  (no_connect (at 121.92 105.41))
-  (no_connect (at 215.9 50.8))
-  (no_connect (at 271.78 107.95))
-  (no_connect (at 121.92 107.95))
-  (no_connect (at 220.98 107.95))
-  (no_connect (at 121.92 48.26))
-  (no_connect (at 121.92 50.8))
-  (no_connect (at 121.92 43.18))
-  (no_connect (at 121.92 45.72))
-  (no_connect (at 170.18 102.87))
   (wire (pts (xy 99.06 95.25) (xy 99.06 97.79))
     (stroke (width 0) (type default) (color 0 0 0 0))
@@
     (pin "1")
     (pin "2")
+  )
+  (symbol (lib_id "Connector:Conn_01x04_Male") (at 172.72 45.72 0) (mirror y) (unit 1)
+    (in_bom yes) (on_board yes) (fields_autoplaced)
+    (property "Reference" "J3" (id 0) (at 173.4312 46.1553 0)
+      (effects (font (size 1.27 1.27)) (justify right))
+    )
+    (property "Value" "Conn_01x04_Male" (id 1) (at 173.4312 48.6922 0)
+      (effects (font (size 1.27 1.27)) (justify right))
+    )
+    (property "Footprint" "" (id 2) (at 172.72 45.72 0)
+      (effects (font (size 1.27 1.27)) hide)
+    )
+    (property "Datasheet" "~" (id 3) (at 172.72 45.72 0)
+      (effects (font (size 1.27 1.27)) hide)
+    )
+    (pin "1")
+    (pin "2")
+    (pin "3")
+    (pin "4")
   )
   (symbol (lib_id "Driver_Motor:Pololu_Breakout_A4988") (at 109.22 105.41 0) (unit 1)
@@
     (pin "1")
   )
+  (symbol (lib_id "Connector:Conn_01x04_Male") (at 127 105.41 0) (mirror y) (unit 1)
+    (in_bom yes) (on_board yes) (fields_autoplaced)
+    (property "Reference" "J6" (id 0) (at 127.7112 105.8453 0)
+      (effects (font (size 1.27 1.27)) (justify right))
+    )
+    (property "Value" "Conn_01x04_Male" (id 1) (at 127.7112 108.3822 0)
+      (effects (font (size 1.27 1.27)) (justify right))
+    )
+    (property "Footprint" "" (id 2) (at 127 105.41 0)
+      (effects (font (size 1.27 1.27)) hide)
+    )
+    (property "Datasheet" "~" (id 3) (at 127 105.41 0)
+      (effects (font (size 1.27 1.27)) hide)
+    )
+    (pin "1")
+    (pin "2")
+    (pin "3")
+    (pin "4")
+  )
   (symbol (lib_id "power:+5V") (at 109.22 27.94 0) (unit 1)
     (in_bom yes) (on_board yes) (fields_autoplaced)
@@
     )
     (pin "1")
+  )
+  (symbol (lib_id "Connector:Conn_01x04_Male") (at 271.78 45.72 0) (mirror y) (unit 1)
+    (in_bom yes) (on_board yes) (fields_autoplaced)
+    (property "Reference" "J5" (id 0) (at 272.4912 46.1553 0)
+      (effects (font (size 1.27 1.27)) (justify right))
+    )
+    (property "Value" "Conn_01x04_Male" (id 1) (at 272.4912 48.6922 0)
+      (effects (font (size 1.27 1.27)) (justify right))
+    )
+    (property "Footprint" "" (id 2) (at 271.78 45.72 0)
+      (effects (font (size 1.27 1.27)) hide)
+    )
+    (property "Datasheet" "~" (id 3) (at 271.78 45.72 0)
+      (effects (font (size 1.27 1.27)) hide)
+    )
+    (pin "1")
+    (pin "2")
+    (pin "3")
+    (pin "4")
   )
   (symbol (lib_id "power:GND") (at 254 68.58 0) (unit 1)
@@
     )
     (pin "1")
+  )
+  (symbol (lib_id "Connector:Conn_01x04_Male") (at 276.86 105.41 0) (mirror y) (unit 1)
+    (in_bom yes) (on_board yes) (fields_autoplaced)
+    (property "Reference" "J9" (id 0) (at 277.5712 105.8453 0)
+      (effects (font (size 1.27 1.27)) (justify right))
+    )
+    (property "Value" "Conn_01x04_Male" (id 1) (at 277.5712 108.3822 0)
+      (effects (font (size 1.27 1.27)) (justify right))
+    )
+    (property "Footprint" "" (id 2) (at 276.86 105.41 0)
+      (effects (font (size 1.27 1.27)) hide)
+    )
+    (property "Datasheet" "~" (id 3) (at 276.86 105.41 0)
+      (effects (font (size 1.27 1.27)) hide)
+    )
+    (pin "1")
+    (pin "2")
+    (pin "3")
+    (pin "4")
   )
   (symbol (lib_id "Device:C_Polarized_US") (at 168.91 233.68 0) (unit 1)
@@
     (pin "9")
   )
+  (symbol (lib_id "Connector:Conn_01x04_Male") (at 220.98 45.72 0) (mirror y) (unit 1)
+    (in_bom yes) (on_board yes) (fields_autoplaced)
+    (property "Reference" "J4" (id 0) (at 221.6912 46.1553 0)
+      (effects (font (size 1.27 1.27)) (justify right))
+    )
+    (property "Value" "Conn_01x04_Male" (id 1) (at 221.6912 48.6922 0)
+      (effects (font (size 1.27 1.27)) (justify right))
+    )
+    (property "Footprint" "" (id 2) (at 220.98 45.72 0)
+      (effects (font (size 1.27 1.27)) hide)
+    )
+    (property "Datasheet" "~" (id 3) (at 220.98 45.72 0)
+      (effects (font (size 1.27 1.27)) hide)
+    )
+    (pin "1")
+    (pin "2")
+    (pin "3")
+    (pin "4")
+  )
   (symbol (lib_id "Driver_Motor:Pololu_Breakout_A4988") (at 203.2 45.72 0) (unit 1)
     (in_bom yes) (on_board yes) (fields_autoplaced)
@@
     )
     (pin "1")
+  )
+  (symbol (lib_id "Connector:Conn_01x04_Male") (at 127 45.72 0) (mirror y) (unit 1)
+    (in_bom yes) (on_board yes) (fields_autoplaced)
+    (property "Reference" "J2" (id 0) (at 127.7112 46.1553 0)
+      (effects (font (size 1.27 1.27)) (justify right))
+    )
+    (property "Value" "" (id 1) (at 127.7112 48.6922 0)
+      (effects (font (size 1.27 1.27)) (justify right))
+    )
+    (property "Footprint" "" (id 2) (at 127 45.72 0)
+      (effects (font (size 1.27 1.27)) hide)
+    )
+    (property "Datasheet" "~" (id 3) (at 127 45.72 0)
+      (effects (font (size 1.27 1.27)) hide)
+    )
+    (pin "1")
+    (pin "2")
+    (pin "3")
+    (pin "4")
   )
   (symbol (lib_id "Device:C_Polarized_US") (at 189.23 233.68 0) (unit 1)
@@
     (pin "1")
   )
+  (symbol (lib_id "Connector:Conn_01x04_Male") (at 226.06 105.41 0) (mirror y) (unit 1)
+    (in_bom yes) (on_board yes) (fields_autoplaced)
+    (property "Reference" "J8" (id 0) (at 226.7712 105.8453 0)
+      (effects (font (size 1.27 1.27)) (justify right))
+    )
+    (property "Value" "Conn_01x04_Male" (id 1) (at 226.7712 108.3822 0)
+      (effects (font (size 1.27 1.27)) (justify right))
+    )
+    (property "Footprint" "" (id 2) (at 226.06 105.41 0)
+      (effects (font (size 1.27 1.27)) hide)
+    )
+    (property "Datasheet" "~" (id 3) (at 226.06 105.41 0)
+      (effects (font (size 1.27 1.27)) hide)
+    )
+    (pin "1")
+    (pin "2")
+    (pin "3")
+    (pin "4")
+  )
   (symbol (lib_id "Driver_Motor:Pololu_Breakout_A4988") (at 157.48 105.41 0) (unit 1)
     (in_bom yes) (on_board yes) (fields_autoplaced)
@@
     (pin "1")
   )
+  (symbol (lib_id "Connector:Conn_01x04_Male") (at 175.26 105.41 0) (mirror y) (unit 1)
+    (in_bom yes) (on_board yes) (fields_autoplaced)
+    (property "Reference" "J7" (id 0) (at 175.9712 105.8453 0)
+      (effects (font (size 1.27 1.27)) (justify right))
+    )
+    (property "Value" "Conn_01x04_Male" (id 1) (at 175.9712 108.3822 0)
+      (effects (font (size 1.27 1.27)) (justify right))
+    )
+    (property "Footprint" "" (id 2) (at 175.26 105.41 0)
+      (effects (font (size 1.27 1.27)) hide)
+    )
+    (property "Datasheet" "~" (id 3) (at 175.26 105.41 0)
+      (effects (font (size 1.27 1.27)) hide)
+    )
+    (pin "1")
+    (pin "2")
+    (pin "3")
+    (pin "4")
+  )
   (sheet_instances
     (path "/" (page "1"))
@@
       (reference "J1") (unit 1) (value "MEC2-30-01-X-TH1-NP-WT") (footprint "LIBRARIES:MEC2-30-01-J-TH1-NP-WT-EDGECARD")
     )
-  )
+    (path "/abd5b1f8-417b-4e4b-bb91-50def48c6e7b"
+      (reference "J2") (unit 1) (value "Conn_01x04_Male") (footprint "Connector_PinHeader_2.54mm:PinHeader_1x04_P2.54mm_Vertical")
+    )
+    (path "/0c2f3eaf-b3e7-4140-8945-a10b3c90c28a"
+      (reference "J3") (unit 1) (value "Conn_01x04_Male") (footprint "Connector_PinHeader_2.54mm:PinHeader_1x04_P2.54mm_Vertical")
+    )
+    (path "/6eea4de7-227d-40d6-acc1-1620ef137fa5"
+      (reference "J4") (unit 1) (value "Conn_01x04_Male") (footprint "Connector_PinHeader_2.54mm:PinHeader_1x04_P2.54mm_Vertical")
+    )
+    (path "/2157c811-a41c-4413-a686-7eeaf715ac77"
+      (reference "J5") (unit 1) (value "Conn_01x04_Male") (footprint "Connector_PinHeader_2.54mm:PinHeader_1x04_P2.54mm_Vertical")
+    )
+    (path "/1b2913a9-3614-49e9-ab61-b0b56b565983"
+      (reference "J6") (unit 1) (value "Conn_01x04_Male") (footprint "Connector_PinHeader_2.54mm:PinHeader_1x04_P2.54mm_Vertical")
+    )
+    (path "/ff48192e-40b0-4411-96e4-2f900d824e31"
+      (reference "J7") (unit 1) (value "Conn_01x04_Male") (footprint "Connector_PinHeader_2.54mm:PinHeader_1x04_P2.54mm_Vertical")
+    )
+    (path "/d7624cde-c6c6-4d03-ac2b-041d0cce66db"
+      (reference "J8") (unit 1) (value "Conn_01x04_Male") (footprint "Connector_PinHeader_2.54mm:PinHeader_1x04_P2.54mm_Vertical")
+    )
+    (path "/5f92ba12-4eb5-42c9-af9e-43475b75c780"
+      (reference "J9") (unit 1) (value "Conn_01x04_Male") (footprint "Connector_PinHeader_2.54mm:PinHeader_1x04_P2.54mm_Vertical")
+    )
+  )
