File: PCB/32-STEPPER-DRIVER-BOARD/32-STEPPER-DRIVER-BOARD.kicad_pcb (KiCad board)
At the start: 4 copper layers, 100 x 102.8 mm, 346 parts, among them J1 MEC2-30-01-X-TH1-NP-WT, J2 MEC2-30-01-X-TH1-NP-WT, J3 MEC2-30-01-X-TH1-NP-WT, J4 MEC2-30-01-X-TH1-NP-WT, J5 IPS1-125-01-S-D, J6 UMPT-06-01-X-RA-WT-P-X, U1 74HC595, U10 74HC595, U11 74HC595, U12 74HC595, U13 74HC595, U14 74HC595, U15 74HC595, U16 74HC595, U17 74HC595, U18 74HC595, U19 74HC595, U2 74HC595, U20 74HC595, U21 74HC595, U3 74HC595, U4 74HC595, U5 74HC595, U6 74HC595, U7 74HC595, U9 74HC595

Commit message: cleanup before DRC Errors
Parts:
- added JP1: SolderJumper_2_Open, Jumper:SolderJumper-2_P1.3mm_Open_RoundedPad1.0x1.5mm, F.Cu at (59.9, 33.7)
- added JP2: SolderJumper_2_Open, Jumper:SolderJumper-2_P1.3mm_Open_RoundedPad1.0x1.5mm, F.Cu at (59.9, 83.7)
- J6: moved to F.Cu
- moved J6 108.3 mm to (151.4, 99.0)
- moved J5 18.4 mm to (151.4, 54.4)
- moved U16 1.71 mm to (78.1, 80.1)
- moved U14 1.68 mm to (94.1, 80.1)
- moved U15 1.63 mm to (86.1, 80.1)
- moved U17 1.56 mm to (110.1, 105.2)
- moved U18 1.41 mm to (102.1, 105.2)
- moved U19 1.41 mm to (94.1, 105.2)
- moved U20 1.41 mm to (86.1, 105.2)
- moved U21 1.41 mm to (78.1, 105.2)
- moved D100 1.39 mm to (111.8, 80.0)
- moved D102 1.39 mm to (108.8, 79.9)
- moved D103 1.39 mm to (105.8, 79.9)
- moved D104 1.39 mm to (102.8, 79.9)
- moved D105 1.39 mm to (99.8, 79.9)
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Connections:
- J5 pad 33: unconnected-(J5-Pad33) -> SER1
- J5 pad 34: unconnected-(J5-Pad34) -> SRCLK1
- J5 pad 35: unconnected-(J5-Pad35) -> SRCLK2
- J5 pad 36: unconnected-(J5-Pad36) -> ~{SRCLR}
- J5 pad 37: unconnected-(J5-Pad37) -> ~{OE}
- J5 pad 38: unconnected-(J5-Pad38) -> RCLK
- J5 pad 39: unconnected-(J5-Pad39) -> SRCLK3
- J5 pad 40: unconnected-(J5-Pad40) -> SER2
- J5 pad 41: unconnected-(J5-Pad41) -> SRCLK4
- J5 pad 42: unconnected-(J5-Pad42) -> SER3
- J5 pad 44: unconnected-(J5-Pad44) -> SER4
- J6 pad 02: VCC -> GND
- J6 pad 05: GND -> VCC
- R1 pad 2: GND -> GND1
- R10 pad 2: GND -> GND1
- R100 pad 2: GND -> GND2
- R102 pad 2: GND -> GND2
- R103 pad 2: GND -> GND2
- R104 pad 2: GND -> GND2
- R105 pad 2: GND -> GND2
- R106 pad 2: GND -> GND2
- R108 pad 2: GND -> GND2
- R109 pad 2: GND -> GND2
- R110 pad 2: GND -> GND2
- R111 pad 2: GND -> GND2
- R112 pad 2: GND -> GND2
- R114 pad 2: GND -> GND2
- R115 pad 2: GND -> GND2
- R116 pad 2: GND -> GND2
- R117 pad 2: GND -> GND2
- R118 pad 2: GND -> GND2
- R12 pad 2: GND -> GND1
- R120 pad 2: GND -> GND2
- R121 pad 2: GND -> GND2
- R123 pad 2: GND -> GND2
- R124 pad 2: GND -> GND2
- R125 pad 2: GND -> GND2
- R126 pad 2: GND -> GND2
- R127 pad 2: GND -> GND2
- R129 pad 2: GND -> GND2
- R13 pad 2: GND -> GND1
- R130 pad 2: GND -> GND2
- R131 pad 2: GND -> GND2
- R132 pad 2: GND -> GND2
- R133 pad 2: GND -> GND2
- R135 pad 2: GND -> GND2
- R136 pad 2: GND -> GND2
- R137 pad 2: GND -> GND2
- R138 pad 2: GND -> GND2
- R139 pad 2: GND -> GND2
- R14 pad 2: GND -> GND1
- R141 pad 2: GND -> GND2
- R142 pad 2: GND -> GND2
- R143 pad 2: GND -> GND2
- R144 pad 2: GND -> GND2
- R145 pad 2: GND -> GND2
- R146 pad 2: GND -> GND2
- R147 pad 2: GND -> GND2
- R148 pad 2: GND -> GND2
- R15 pad 2: GND -> GND1
- R150 pad 2: GND -> GND2
- R151 pad 2: GND -> GND2
- R152 pad 2: GND -> GND2
- R153 pad 2: GND -> GND2
- R154 pad 2: GND -> GND2
- R156 pad 2: GND -> GND2
- R157 pad 2: GND -> GND2
- R158 pad 2: GND -> GND2
- R159 pad 2: GND -> GND2
- R16 pad 2: GND -> GND1
- R160 pad 2: GND -> GND2
- R162 pad 2: GND -> GND2
- R163 pad 2: GND -> GND2
- R164 pad 2: GND -> GND2
- R165 pad 2: GND -> GND2
- R166 pad 2: GND -> GND2
- R168 pad 2: GND -> GND2
- R169 pad 2: GND -> GND2
- R170 pad 2: GND -> GND2
- R171 pad 2: GND -> GND2
- R172 pad 2: GND -> GND2
- R174 pad 2: GND -> GND2
- R175 pad 2: GND -> GND2
- R176 pad 2: GND -> GND2
- R177 pad 2: GND -> GND2
- R178 pad 2: GND -> GND2
- R18 pad 2: GND -> GND1
- R180 pad 2: GND -> GND2
- R181 pad 2: GND -> GND2
- R182 pad 2: GND -> GND2
- R183 pad 2: GND -> GND2
- R184 pad 2: GND -> GND2
- R186 pad 2: GND -> GND2
- R187 pad 2: GND -> GND2
- R188 pad 2: GND -> GND2
- R189 pad 2: GND -> GND2
- R19 pad 2: GND -> GND1
- R190 pad 2: GND -> GND2
- R192 pad 2: GND -> GND2
- R2 pad 2: GND -> GND1
- R20 pad 2: GND -> GND1
- R21 pad 2: GND -> GND1
- R22 pad 2: GND -> GND1
- R24 pad 2: GND -> GND1
- R25 pad 2: GND -> GND1
- R27 pad 2: GND -> GND1
- R28 pad 2: GND -> GND1
- R29 pad 2: GND -> GND1
- R3 pad 2: GND -> GND1
- R30 pad 2: GND -> GND1
- R31 pad 2: GND -> GND1
- R33 pad 2: GND -> GND1
- R34 pad 2: GND -> GND1
- R35 pad 2: GND -> GND1
- R36 pad 2: GND -> GND1
- R37 pad 2: GND -> GND1
- R39 pad 2: GND -> GND1
- R4 pad 2: GND -> GND1
- R40 pad 2: GND -> GND1
- R41 pad 2: GND -> GND1
- R42 pad 2: GND -> GND1
- R43 pad 2: GND -> GND1
- R45 pad 2: GND -> GND1
- R46 pad 2: GND -> GND1
- R47 pad 2: GND -> GND1
- R48 pad 2: GND -> GND1
- R49 pad 2: GND -> GND1
- R50 pad 2: GND -> GND1
- R51 pad 2: GND -> GND1
- R52 pad 2: GND -> GND1
- R54 pad 2: GND -> GND1
- R55 pad 2: GND -> GND1
- R56 pad 2: GND -> GND1
- R57 pad 2: GND -> GND1
- R58 pad 2: GND -> GND1
- R6 pad 2: GND -> GND1
- R60 pad 2: GND -> GND1
- R61 pad 2: GND -> GND1
- R62 pad 2: GND -> GND1
- R63 pad 2: GND -> GND1
- R64 pad 2: GND -> GND1
- R66 pad 2: GND -> GND1
- R67 pad 2: GND -> GND1
- R68 pad 2: GND -> GND1
- R69 pad 2: GND -> GND1
- R7 pad 2: GND -> GND1
- R70 pad 2: GND -> GND1
- R72 pad 2: GND -> GND1
- R73 pad 2: GND -> GND1
- R75 pad 2: GND -> GND1
- R76 pad 2: GND -> GND1
- R77 pad 2: GND -> GND1
- R78 pad 2: GND -> GND1
- R79 pad 2: GND -> GND1
- R8 pad 2: GND -> GND1
- R81 pad 2: GND -> GND1
- R82 pad 2: GND -> GND1
- R83 pad 2: GND -> GND1
- R84 pad 2: GND -> GND1
- R85 pad 2: GND -> GND1
- R87 pad 2: GND -> GND1
- R88 pad 2: GND -> GND1
- R89 pad 2: GND -> GND1
- R9 pad 2: GND -> GND1
- R90 pad 2: GND -> GND1
- R91 pad 2: GND -> GND1
- R93 pad 2: GND -> GND1
- R94 pad 2: GND -> GND1
- R95 pad 2: GND -> GND1
- R96 pad 2: GND -> GND1
- R97 pad 2: GND -> GND2
- R98 pad 2: GND -> GND2
- R99 pad 2: GND -> GND2
- U1 pad 11: SRCLK -> SRCLK1
- U10 pad 11: SRCLK -> SRCLK2
- U11 pad 11: SRCLK -> SRCLK2
- U12 pad 11: SRCLK -> SRCLK3
- U13 pad 1: 3A7MS2 -> 3A7MS1
- U13 pad 11: SRCLK -> SRCLK3
- U13 pad 15: 3A3MS2 -> 3A3MS1
- U13 pad 2: 3A3MS3 -> 3A3MS2
- U13 pad 3: 3A7MS3 -> 3A7MS2
- U13 pad 4: 3DIR4 -> 3A3MS3
- U13 pad 5: 3DIR8 -> 3A7MS3
- U13 pad 6: 3DIR3 -> 3DIR4
- U13 pad 7: 3DIR7 -> 3DIR8
- U14 pad 1: 3A7EN -> 3A6MS2
- U14 pad 11: SRCLK -> SRCLK3
- U14 pad 15: 3A3EN -> 3A2MS2
- U14 pad 2: 3A3MS1 -> 3A2MS3
- U14 pad 3: 3A7MS1 -> 3A6MS3
- U14 pad 4: 3A1MS2 -> 3DIR3
- U14 pad 5: 3A5MS2 -> 3DIR7
- U14 pad 6: 3A1MS3 -> 3A3EN
- U14 pad 7: 3A5MS3 -> 3A7EN
- U15 pad 1: 3A6MS3 -> 3A5MS3
- U15 pad 11: SRCLK -> SRCLK3
- U15 pad 15: 3A2MS3 -> 3A1MS3
- U15 pad 2: 3DIR1 -> 3DIR2
- U15 pad 3: 3DIR5 -> 3DIR6
- U15 pad 4: 3A1EN -> 3A2EN
- U15 pad 5: 3A5EN -> 3A6EN
- U15 pad 6: 3A1MS1 -> 3A2MS1
- U15 pad 7: 3A5MS1 -> 3A6MS1
- U15 pad 9: unconnected-(U15-Pad9) -> Net-(U16-Pad14)
- U16 pad 1: 3DIR6 -> 3DIR5
- U16 pad 11: SRCLK -> SRCLK3
- U16 pad 14: unconnected-(U16-Pad14) -> Net-(U16-Pad14)
- U16 pad 15: 3DIR2 -> 3DIR1
- U16 pad 2: 3A2EN -> 3A1EN
- U16 pad 3: 3A6EN -> 3A5EN
- U16 pad 4: 3A2MS1 -> 3A1MS1
- U16 pad 5: 3A6MS1 -> 3A5MS1
- U16 pad 6: 3A2MS2 -> 3A1MS2
- U16 pad 7: 3A6MS2 -> 3A5MS2
- U17 pad 11: SRCLK -> SRCLK4
- U18 pad 1: 4A7MS2 -> 4A7MS1
- U18 pad 11: SRCLK -> SRCLK4
- U18 pad 15: 4A3MS2 -> 4A3MS1
- U18 pad 2: 4A3MS3 -> 4A3MS2
- U18 pad 3: 4A7MS3 -> 4A7MS2
- U18 pad 4: 4DIR4 -> 4A3MS3
- U18 pad 5: 4DIR8 -> 4A7MS3
- U18 pad 6: 4DIR3 -> 4DIR4
- U18 pad 7: 4DIR7 -> 4DIR8
- U19 pad 1: 4A7EN -> 4A6MS2
- U19 pad 11: SRCLK -> SRCLK4
- U19 pad 15: 4A3EN -> 4A2MS2
- U19 pad 2: 4A3MS1 -> 4A2MS3
- U19 pad 3: 4A7MS1 -> 4A6MS3
- U19 pad 4: 4A2EN -> 4DIR3
- U19 pad 5: 4A6EN -> 4DIR7
- U19 pad 6: 4A2MS1 -> 4A3EN
- U19 pad 7: 4A6MS1 -> 4A7EN
- U2 pad 11: SRCLK -> SRCLK1
- U20 pad 1: 4A6MS2 -> 4A5MS3
- U20 pad 11: SRCLK -> SRCLK4
- U20 pad 15: 4A2MS2 -> 4A1MS3
- U20 pad 2: 4A2MS3 -> 4DIR2
- U20 pad 3: 4A6MS3 -> 4DIR6
- U20 pad 4: 4A1MS2 -> 4A2EN
- U20 pad 5: 4A5MS2 -> 4A6EN
- U20 pad 6: 4A1MS3 -> 4A2MS1
- U20 pad 7: 4A5MS3 -> 4A6MS1
- U21 pad 1: 4DIR6 -> 4DIR5
- U21 pad 11: SRCLK -> SRCLK4
- U21 pad 15: 4DIR2 -> 4DIR1
- U21 pad 2: 4DIR1 -> 4A1EN
- U21 pad 3: 4DIR5 -> 4A5EN
- U21 pad 4: 4A1EN -> 4A1MS1
- U21 pad 5: 4A5EN -> 4A5MS1
- U21 pad 6: 4A1MS1 -> 4A1MS2
- U21 pad 7: 4A5MS1 -> 4A5MS2
- U3 pad 11: SRCLK -> SRCLK1
- U4 pad 11: SRCLK -> SRCLK1
- U5 pad 11: SRCLK -> SRCLK1
- U6 pad 11: SRCLK -> SRCLK2
- U7 pad 11: SRCLK -> SRCLK2
- U9 pad 11: SRCLK -> SRCLK2
Routing:
- net GND: track 0.00 -> 510.3 mm, vias 0 -> 63
- net ~{OE}: track 197.0 -> 415.0 mm, vias 0 -> 24
- net RCLK: track 195.0 -> 395.1 mm, vias 0 -> 24
- net SRCLK: track 194.0 -> 0.00 mm
- net +5V: track 198.7 -> 379.6 mm, vias 0 -> 28
- net ~{SRCLR}: track 192.0 -> 365.6 mm, vias 0 -> 24
- net GND1: track 0.00 -> 158.1 mm
- net GND2: track 0.00 -> 157.0 mm
- net SRCLK4: track 0.00 -> 121.7 mm, vias 0 -> 7
- net SRCLK1: track 0.00 -> 118.0 mm, vias 0 -> 5
- net SRCLK3: track 0.00 -> 101.6 mm, vias 0 -> 5
- net SRCLK2: track 0.00 -> 98.4 mm, vias 0 -> 5
- net SER1: track 0.00 -> 75.0 mm, vias 0 -> 1
- net SER4: track 0.00 -> 73.9 mm, vias 0 -> 1
- net SER3: track 0.00 -> 53.9 mm, vias 0 -> 1
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- added copper zone on B.Cu, net +5V
- added copper zone on F.Cu, net +5V
- added copper zone on F.Cu, net GND
- added copper zone on In2.Cu, net GND
- added copper zone on F.Cu, net VCC
- added copper zone on In1.Cu, net VCC
- removed copper zone on B.Cu, net VCC
Other:
- board size 100 x 102.8 mm -> 115 x 102.8 mm
- board text added: "A1EN"
- board text added: "A1MS1"
- board text added: "A1MS2"
- board text added: "A1MS3"
- board text added: "A2EN"
- board text added: "A2MS1"
- board text added: "A2MS2"
- board text added: "A2MS3"
- board text added: "A3EN"
- board text added: "A3MS1"
- board text added: "A3MS2"
- board text added: "A3MS3"
- board text added: "A4EN"
- board text added: "A4MS1"
- board text added: "A4MS2"
- board text added: "A4MS3"
- board text added: "A5EN"
- board text added: "A5MS1"
- board text added: "A5MS2"
- board text added: "A5MS3"
- board text added: "A6EN"
- board text added: "A6MS1"
- board text added: "A6MS2"
- board text added: "A6MS3"
- board text added: "A7EN"
- board text added: "A7MS1"
- board text added: "A7MS2"
- board text added: "A7MS3"
- board text added: "A8EN"
- board text added: "A8MS1"
- board text added: "A8MS2"
- board text added: "A8MS3"
- board text added: "DIR1"
- board text added: "DIR2"
- board text added: "DIR3"
- board text added: "DIR4"
- board text added: "DIR5"
- board text added: "DIR6"
- board text added: "DIR7"
- board text added: "DIR8"
- board text removed: "1A1EN"
- board text removed: "1A1MS1"
- board text removed: "1A1MS2"
- board text removed: "1A1MS3"
- board text removed: "1A2EN"
- board text removed: "1A2MS1"
- board text removed: "1A2MS2"
- board text removed: "1A2MS3"
- board text removed: "1A3EN"
- board text removed: "1A3MS1"
- board text removed: "1A3MS2"
- board text removed: "1A3MS3"
- board text removed: "1A4EN"
- board text removed: "1A4MS1"
- board text removed: "1A4MS2"
- board text removed: "1A4MS3"
- board text removed: "1A5EN"
- board text removed: "1A5MS1"
- board text removed: "1A5MS2"
- board text removed: "1A5MS3"
- board text removed: "1A6EN"
- board text removed: "1A6MS1"
- board text removed: "1A6MS2"
- board text removed: "1A6MS3"
- board text removed: "1A7EN"
- board text removed: "1A7MS1"
- board text removed: "1A7MS2"
- board text removed: "1A7MS3"
- board text removed: "1A8EN"
- board text removed: "1A8MS1"
- board text removed: "1A8MS2"
- board text removed: "1A8MS3"
- board text removed: "1DIR1"
- board text removed: "1DIR2"
- board text removed: "1DIR3"
- board text removed: "1DIR4"
- board text removed: "1DIR5"
- board text removed: "1DIR6"
- board text removed: "1DIR7"
- board text removed: "1DIR8"
- board text removed: "2DIR1"

Commit message: Final checks for 32-stepper driver
Routing:
- added copper zone on B.Cu, net GND
- added copper zone on In1.Cu, net GND

Commit message: generate gerber for price check
Other:
- board text added: "32-STEPPER-DRIVER-BOARD REV A ELLIOT EICKHOLTZ"
Changed lines of the file:
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@@
       (outputformat 1)
       (mirror false)
-      (drillshape 1)
+      (drillshape 0)
       (scaleselection 1)
       (outputdirectory "")
@@
     (pad "S3" thru_hole circle (at 9.55 -1 90) (size 1.308 1.308) (drill 0.8) (layers *.Cu *.Mask))
     (pad "S4" thru_hole circle (at 9.55 1 90) (size 1.308 1.308) (drill 0.8) (layers *.Cu *.Mask))
-    (model "C:/Users/34892/OneDrive - Samtec/Documents/GitHub/64-Stepper-Motor-Controller/PCB/LIBRARIES/UMPT-06-01-X-RA-WT-P-X.step"
+    (model "${LOCAL}/UMPT-06-01-X-RA-WT-P-X.step"
       (offset (xyz 0 -2.25 0))
       (scale (xyz 1 1 1))
@@
     (pad "S1" thru_hole circle (at -32.7 0) (size 1.508 1.508) (drill 1) (layers *.Cu *.Mask))
     (pad "S2" thru_hole circle (at 32.7 0) (size 1.508 1.508) (drill 1) (layers *.Cu *.Mask))
-    (model "C:/Users/34892/OneDrive - Samtec/Documents/GitHub/64-Stepper-Motor-Controller/PCB/LIBRARIES/8-STEPPER-CARD-ASSEMBLY v3.step"
+    (model "${LOCAL}/8-STEPPER-CARD-ASSEMBLY v3.step"
       (offset (xyz -158.75 0.75 123))
       (scale (xyz 1 1 1))
@@
     (pad "S1" thru_hole circle (at -32.7 0) (size 1.508 1.508) (drill 1) (layers *.Cu *.Mask))
     (pad "S2" thru_hole circle (at 32.7 0) (size 1.508 1.508) (drill 1) (layers *.Cu *.Mask))
-    (model "C:/Users/34892/OneDrive - Samtec/Documents/GitHub/64-Stepper-Motor-Controller/PCB/LIBRARIES/8-STEPPER-CARD-ASSEMBLY v3.step"
+    (model "${LOCAL}/8-STEPPER-CARD-ASSEMBLY v3.step"
       (offset (xyz -158 0.75 123))
       (scale (xyz 1 1 1))
@@
     (pad "S1" thru_hole circle (at -32.7 0) (size 1.508 1.508) (drill 1) (layers *.Cu *.Mask))
     (pad "S2" thru_hole circle (at 32.7 0) (size 1.508 1.508) (drill 1) (layers *.Cu *.Mask))
-    (model "C:/Users/34892/OneDrive - Samtec/Documents/GitHub/64-Stepper-Motor-Controller/PCB/LIBRARIES/8-STEPPER-CARD-ASSEMBLY v3.step"
+    (model "${LOCAL}/8-STEPPER-CARD-ASSEMBLY v3.step"
       (offset (xyz -158.75 0.75 123))
       (scale (xyz 1 1 1))
@@
     (pad "S1" thru_hole circle (at -32.7 0) (size 1.508 1.508) (drill 1) (layers *.Cu *.Mask))
     (pad "S2" thru_hole circle (at 32.7 0) (size 1.508 1.508) (drill 1) (layers *.Cu *.Mask))
-    (model "C:/Users/34892/OneDrive - Samtec/Documents/GitHub/64-Stepper-Motor-Controller/PCB/LIBRARIES/8-STEPPER-CARD-ASSEMBLY v3.step"
+    (model "${LOCAL}/8-STEPPER-CARD-ASSEMBLY v3.step"
       (offset (xyz -158.75 0.75 123))
       (scale (xyz 1 1 1))
@@
     (pad "50" thru_hole circle locked (at -30.48 -1.27 90) (size 1.39 1.39) (drill 1.04) (layers *.Cu *.Mask)
       (net 376 "unconnected-(J5-Pad50)") (pinfunction "50") (pintype "passive"))
-    (model "C:/Users/34892/OneDrive - Samtec/Documents/GitHub/64-Stepper-Motor-Controller/PCB/LIBRARIES/IPT1-125-01-S-D.step"
+    (model "${LOCAL}/IPT1-125-01-S-D.step"
       (offset (xyz 0 0 0))
       (scale (xyz 1 1 1))
@@
     (effects (font (size 1 1) (thickness 0.15)))
   )
+  (gr_text "32-STEPPER-DRIVER-BOARD REV A\nELLIOT EICKHOLTZ" (at 141.4272 55.2196 90) (layer "F.SilkS")
+    (effects (font (size 1 1) (thickness 0.15)))
+  )
   (gr_text "DIR6" (at 80.381 26.516 90) (layer "F.SilkS")
     (effects (font (size 1 1) (thickness 0.15)))
@@
   (via (at 42.926 115.189) (size 0.45) (drill 0.2) (layers "F.Cu" "B.Cu") (free) (net 1))
   (via (at 152.019 98.552) (size 0.45) (drill 0.2) (layers "F.Cu" "B.Cu") (free) (net 1))
-  (via (at 127.127 18.161) (size 0.45) (drill 0.2) (layers "F.Cu" "B.Cu") (free) (net 1))
+  (via (at 126.2126 18.161) (size 0.45) (drill 0.2) (layers "F.Cu" "B.Cu") (free) (net 1))
   (via (at 148.971 102.616) (size 0.45) (drill 0.2) (layers "F.Cu" "B.Cu") (free) (net 1))
   (via (at 58.039 98.679) (size 0.45) (drill 0.2) (layers "F.Cu" "B.Cu") (free) (net 1))
   (via (at 151.003 93.345) (size 0.45) (drill 0.2) (layers "F.Cu" "B.Cu") (free) (net 1))
-  (via (at 151.257 18.288) (size 0.45) (drill 0.2) (layers "F.Cu" "B.Cu") (free) (net 1))
+  (via (at 142.7734 18.161) (size 0.45) (drill 0.2) (layers "F.Cu" "B.Cu") (free) (net 1))
   (via (at 148.971 94.615) (size 0.45) (drill 0.2) (layers "F.Cu" "B.Cu") (free) (net 1))
   (via (at 49.657 17.653) (size 0.45) (drill 0.2) (layers "F.Cu" "B.Cu") (free) (net 1))
@@
   (via (at 151.003 94.615) (size 0.45) (drill 0.2) (layers "F.Cu" "B.Cu") (free) (net 1))
   (via (at 43.434 82.169) (size 0.45) (drill 0.2) (layers "F.Cu" "B.Cu") (free) (net 1))
-  (via (at 130.302 18.161) (size 0.45) (drill 0.2) (layers "F.Cu" "B.Cu") (free) (net 1))
+  (via (at 129.3876 18.161) (size 0.45) (drill 0.2) (layers "F.Cu" "B.Cu") (free) (net 1))
   (via (at 149.987 93.345) (size 0.45) (drill 0.2) (layers "F.Cu" "B.Cu") (free) (net 1))
   (via (at 50.038 82.169) (size 0.45) (drill 0.2) (layers "F.Cu" "B.Cu") (free) (net 1))
@@
   (via (at 45.847 30.353) (size 0.45) (drill 0.2) (layers "F.Cu" "B.Cu") (free) (net 1))
   (via (at 152.019 101.346) (size 0.45) (drill 0.2) (layers "F.Cu" "B.Cu") (free) (net 1))
-  (via (at 144.653 18.288) (size 0.45) (drill 0.2) (layers "F.Cu" "B.Cu") (free) (net 1))
+  (via (at 136.1694 18.161) (size 0.45) (drill 0.2) (layers "F.Cu" "B.Cu") (free) (net 1))
   (via (at 57.912 74.041) (size 0.45) (drill 0.2) (layers "F.Cu" "B.Cu") (free) (net 1))
   (via (at 43.307 47.752) (size 0.45) (drill 0.2) (layers "F.Cu" "B.Cu") (free) (net 1))
@@
   (via (at 149.987 97.282) (size 0.45) (drill 0.2) (layers "F.Cu" "B.Cu") (free) (net 1))
   (via (at 58.039 105.283) (size 0.45) (drill 0.2) (layers "F.Cu" "B.Cu") (free) (net 1))
-  (via (at 133.731 18.161) (size 0.45) (drill 0.2) (layers "F.Cu" "B.Cu") (free) (net 1))
+  (via (at 132.8166 18.161) (size 0.45) (drill 0.2) (layers "F.Cu" "B.Cu") (free) (net 1))
   (via (at 43.307 99.568) (size 0.45) (drill 0.2) (layers "F.Cu" "B.Cu") (free) (net 1))
   (via (at 46.482 47.752) (size 0.45) (drill 0.2) (layers "F.Cu" "B.Cu") (free) (net 1))
-  (via (at 147.828 18.288) (size 0.45) (drill 0.2) (layers "F.Cu" "B.Cu") (free) (net 1))
+  (via (at 139.3444 18.161) (size 0.45) (drill 0.2) (layers "F.Cu" "B.Cu") (free) (net 1))
   (via (at 148.971 98.552) (size 0.45) (drill 0.2) (layers "F.Cu" "B.Cu") (free) (net 1))
   (via (at 46.101 115.189) (size 0.45) (drill 0.2) (layers "F.Cu" "B.Cu") (free) (net 1))

Commit message: final adjustments
Parts:
- added J10: Screw_Terminal_01x01, MountingHole:MountingHole_2.2mm_M2_Pad, F.Cu at (151.8, 114.3)
- added J7: Screw_Terminal_01x01, MountingHole:MountingHole_2.2mm_M2_Pad, F.Cu at (44.5, 19.1)
- added J8: Screw_Terminal_01x01, MountingHole:MountingHole_2.2mm_M2_Pad, F.Cu at (151.8, 19.1)
- added J9: Screw_Terminal_01x01, MountingHole:MountingHole_2.2mm_M2_Pad, F.Cu at (44.5, 114.3)
Connections:
- J5 pad 43: unconnected-(J5-Pad43) -> VCC
- J5 pad 45: unconnected-(J5-Pad45) -> +5V
- J5 pad 46: unconnected-(J5-Pad46) -> +5V
- J5 pad 47: unconnected-(J5-Pad47) -> GND
- J5 pad 48: unconnected-(J5-Pad48) -> GND
- J5 pad 49: unconnected-(J5-Pad49) -> GND
- J5 pad 50: unconnected-(J5-Pad50) -> GND
Routing:
- net +5V: track 379.6 -> 415.0 mm
- net VCC: track 0.00 -> 26.1 mm
- net GND: vias 63 -> 57
