File: PCB/32-STEPPER-DRIVER-BOARD/32-STEPPER-DRIVER-BOARD.kicad_sch (KiCad schematic)
At the start: 28 parts

Commit message: begin 32 stepper board
Parts:
- J?: value (none) -> MEC2-30-01-X-TH1-NP-WT; footprint (none) -> SAMTEC_MEC2-30-01-X-TH1-NP-WT
Connections:
- net GND: now reaches J?.01
- net GND: now also J?.01, J?.01, J?.01, J?.02, J?.02, J?.02, J?.02, J?.03, J?.03, J?.03, J?.03, J?.04, J?.04, J?.04, J?.04
- net VCC: now reaches J?.05
- net VCC: now also J?.05, J?.05, J?.05, J?.06, J?.06, J?.06, J?.06, J?.07, J?.07, J?.07, J?.07, J?.08, J?.08, J?.08, J?.08, J?.09, J?.09, J?.09, J?.09, J?.10, J?.10, J?.10, J?.10
- net +5V: now reaches J?.59
- net +5V: now also J?.59, J?.59, J?.59, J?.60, J?.60, J?.60, J?.60

Commit message: initial 32-driver layout
Parts:
- added D1: (no value), symbol Device:LED
- added D10, D100, D101, D102, D103, D104, D105, D106, D107, D108, D109, D11, D110, D111, D112, D113, D114, D115, D116, D117, D118, D119, D12, D120, D121, D122, D123, D124, D125, D126, D127, D128, D129, D13, D130, D131, D132, D133, D134, D135, D136, D137, D138, D139, D14, D140, D141, D142, D143, D144, D145, D146, D147, D148, D149, D15, D150, D151, D152, D153, D154, D155, D156, D157, D158, D159, D16, D160, D161, D162, D163, D164, D165, D166, D167, D168, D169, D17, D170, D171, D172, D173, D174, D175, D176, D177, D178, D179, D18, D180, D181, D182, D183, D184, D185, D186, D187, D188, D189, D19, D190, D191, D192, D2, D20, D21, D22, D23, D24, D25, D26, D27, D28, D29, D3, D30, D31, D32, D33, D34, D35, D36, D37, D38, D39, D4, D40, D41, D42, D43, D44, D45, D46, D47, D48, D49, D5, D50, D51, D52, D53, D54, D55, D56, D57, D58, D59, D6, D60, D61, D62, D63, D64, D65, D66, D67, D68, D69, D7, D70, D71, D72, D73, D74, D75, D76, D77, D78, D79, D8, D80, D81, D82, D83, D84, D85, D86, D87, D88, D89, D9, D90, D91, D92, D93, D94, D95, D96, D97, D98, D99: LED, symbol Device:LED
- added R1: (no value), symbol Device:R
- added R10, R100, R101, R102, R103, R104, R105, R106, R107, R108, R109, R11, R110, R111, R112, R113, R114, R115, R116, R117, R118, R119, R12, R120, R121, R122, R123, R124, R125, R126, R127, R128, R129, R13, R130, R131, R132, R133, R134, R135, R136, R137, R138, R139, R14, R140, R141, R142, R143, R144, R145, R146, R147, R148, R149, R15, R150, R151, R152, R153, R154, R155, R156, R157, R158, R159, R16, R160, R161, R162, R163, R164, R165, R166, R167, R168, R169, R17, R170, R171, R172, R173, R174, R175, R176, R177, R178, R179, R18, R180, R181, R182, R183, R184, R185, R186, R187, R188, R189, R19, R190, R191, R192, R2, R20, R21, R22, R23, R24, R25, R26, R27, R28, R29, R3, R30, R31, R32, R33, R34, R35, R36, R37, R38, R39, R4, R40, R41, R42, R43, R44, R45, R46, R47, R48, R49, R5, R50, R51, R52, R53, R54, R55, R56, R57, R58, R59, R6, R60, R61, R62, R63, R64, R65, R66, R67, R68, R69, R7, R70, R71, R72, R73, R74, R75, R76, R77, R78, R79, R8, R80, R81, R82, R83, R84, R85, R86, R87, R88, R89, R9, R90, R91, R92, R93, R94, R95, R96, R97, R98, R99: R, symbol Device:R
- J1, J2, J3, J4: renamed from J?; footprint SAMTEC_MEC2-30-01-X-TH1-NP-WT -> (none)
- gave numbers to parts that had none: 24
Connections:
- net +5V: now also U1.16 (VCC), U10.16 (VCC), U11.16 (VCC), U12.16 (VCC), U13.16 (VCC), U14.16 (VCC), U15.16 (VCC), U16.16 (VCC), U17.16 (VCC), U18.16 (VCC), U19.16 (VCC), U2.16 (VCC)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
- net GND: now also U1.8 (GND), U10.8 (GND), U11.8 (GND), U12.8 (GND), U13.8 (GND), U14.8 (GND), U15.8 (GND), U16.8 (GND), U17.8 (GND), U18.8 (GND), U19.8 (GND), U2.8 (GND)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
- net 3DIR5: now reaches U18.1 (QB)
- net 3DIR5: now also J3.12, D121.2 (A)
- net ~{SRCLR}: now reaches U18.10 (~{SRCLR})
- net ~{SRCLR}: now also U1.10 (~{SRCLR}), U10.10 (~{SRCLR}), U11.10 (~{SRCLR}), U12.10 (~{SRCLR}), U13.10 (~{SRCLR}), U14.10 (~{SRCLR}), U15.10 (~{SRCLR}), U16.10 (~{SRCLR}), U17.10 (~{SRCLR}), U19.10 (~{SRCLR}), U2.10 (~{SRCLR}), U20.10 (~{SRCLR})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
- net SRCLK: now reaches U18.11 (SRCLK)
- net SRCLK: now also U1.11 (SRCLK), U10.11 (SRCLK), U11.11 (SRCLK), U12.11 (SRCLK), U13.11 (SRCLK), U14.11 (SRCLK), U15.11 (SRCLK), U16.11 (SRCLK), U17.11 (SRCLK), U19.11 (SRCLK), U2.11 (SRCLK), U20.11 (SRCLK)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
- net RCLK: now reaches U18.12 (RCLK)
- net RCLK: now also U1.12 (RCLK), U10.12 (RCLK), U11.12 (RCLK), U12.12 (RCLK), U13.12 (RCLK), U14.12 (RCLK), U15.12 (RCLK), U16.12 (RCLK), U17.12 (RCLK), U19.12 (RCLK), U2.12 (RCLK), U20.12 (RCLK)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
- net ~{OE}: now reaches U18.13 (~{OE})
- net ~{OE}: now also U1.13 (~{OE}), U10.13 (~{OE}), U11.13 (~{OE}), U12.13 (~{OE}), U13.13 (~{OE}), U14.13 (~{OE}), U15.13 (~{OE}), U16.13 (~{OE}), U17.13 (~{OE}), U19.13 (~{OE}), U2.13 (~{OE}), U20.13 (~{OE})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
- net at U18.14 (SER): now also U17.9 (QH')
- net 3DIR1: now reaches U18.15 (QA)
- net 3DIR1: now also J3.11, D120.2 (A)
- net 3A1STEP: now reaches U18.2 (QC)
- net 3A1STEP: now also J3.13, D119.2 (A)
- net 3A5STEP: now reaches U18.3 (QD)
- net 3A5STEP: now also J3.14, D122.2 (A)
- net 3A1EN: now reaches U18.4 (QE)
- net 3A1EN: now also J3.15, D118.2 (A)
- net 3A5EN: now reaches U18.5 (QF)
- net 3A5EN: now also J3.16, D123.2 (A)
- net 3A1MS1: now reaches U18.6 (QG)
- net 3A1MS1: now also J3.17, D117.2 (A)
- net 3A5MS1: now reaches U18.7 (QH)
- net 3A5MS1: now also J3.18, D124.2 (A)
- net at U18.9 (QH'): now also U19.14 (SER)
- net 1DIR1: now reaches J1.11
- net 1DIR1: now also U6.15 (QA), D24.2 (A)
- net 1DIR5: now reaches J1.12
- net 1DIR5: now also U6.1 (QB), D25.2 (A)
- net 1A1STEP: now reaches J1.13
- net 1A1STEP: now also U6.2 (QC), D23.2 (A)
- net 1A5STEP: now reaches J1.14
- net 1A5STEP: now also U6.3 (QD), D26.2 (A)
- net 1A1EN: now reaches J1.15
- net 1A1EN: now also U6.4 (QE), D22.2 (A)
- net 1A5EN: now reaches J1.16
- net 1A5EN: now also U6.5 (QF), D27.2 (A)
- net 1A1MS1: now reaches J1.17
- net 1A1MS1: now also U6.6 (QG), D21.2 (A)
- net 1A5MS1: now reaches J1.18
- net 1A5MS1: now also U6.7 (QH), D28.2 (A)
- net 1A1MS2: now reaches J1.19
- net 1A1MS2: now also U5.15 (QA), D20.2 (A)
- net 1A5MS2: now reaches J1.20
- net 1A5MS2: now also U5.1 (QB), D29.2 (A)
- net 1A1MS3: now reaches J1.21
- net 1A1MS3: now also U5.2 (QC), D19.2 (A)
- net 1A5MS3: now reaches J1.22
- net 1A5MS3: now also U5.3 (QD), D30.2 (A)
- net 1DIR2: now reaches J1.23
- net 1DIR2: now also U5.4 (QE), D18.2 (A)
- net 1DIR6: now reaches J1.24
- net 1DIR6: now also U5.5 (QF), D31.2 (A)
- net 1A2STEP: now reaches J1.25
- net 1A2STEP: now also U5.6 (QG), D17.2 (A)
- net 1A6STEP: now reaches J1.26
- net 1A6STEP: now also U5.7 (QH), D32.2 (A)
- net 1A2EN: now reaches J1.27
- net 1A2EN: now also U4.15 (QA), D16.2 (A)
- net 1A6EN: now reaches J1.28
- net 1A6EN: now also U4.1 (QB), D33.2 (A)
- net 1A2MS1: now reaches J1.29
- net 1A2MS1: now also U4.2 (QC), D15.2 (A)
- net 1A6MS1: now reaches J1.30
- net 1A6MS1: now also U4.3 (QD), D34.2 (A)
- net 1A2MS2: now reaches J1.31
- net 1A2MS2: now also U4.4 (QE), D14.2 (A)
- net 1A6MS2: now reaches J1.32
- net 1A6MS2: now also U4.5 (QF), D35.2 (A)
- net 1A2MS3: now reaches J1.33
- net 1A2MS3: now also U4.6 (QG), D13.2 (A)
- net 1A6MS3: now reaches J1.34
- net 1A6MS3: now also U4.7 (QH), D36.2 (A)
- net 1DIR3: now reaches J1.35
- net 1DIR3: now also U3.15 (QA), D12.2 (A)
- net 1DIR7: now reaches J1.36
- net 1DIR7: now also U3.1 (QB), D37.2 (A)
- net 1A3STEP: now reaches J1.37
- net 1A3STEP: now also U3.2 (QC), D11.2 (A)
- net 1A7STEP: now reaches J1.38
- net 1A7STEP: now also U3.3 (QD), D38.2 (A)
- net 1A3EN: now reaches J1.39
- net 1A3EN: now also U3.4 (QE), D10.2 (A)
- net 1A7EN: now reaches J1.40
- net 1A7EN: now also U3.5 (QF), D39.2 (A)
- net 1A3MS1: now reaches J1.41
- net 1A3MS1: now also U3.6 (QG), D9.2 (A)
- net 1A7MS1: now reaches J1.42
- net 1A7MS1: now also U3.7 (QH), D40.2 (A)
- net 1A3MS2: now reaches J1.43
- net 1A3MS2: now also U2.15 (QA), D8.2 (A)
- net 1A7MS2: now reaches J1.44
- net 1A7MS2: now also U2.1 (QB), D41.2 (A)
- net 1A3MS3: now reaches J1.45
- net 1A3MS3: now also U2.2 (QC), D7.2 (A)
- net 1A7MS3: now reaches J1.46
- net 1A7MS3: now also U2.3 (QD), D42.2 (A)
- net 1DIR4: now reaches J1.47
- net 1DIR4: now also U2.4 (QE), D6.2 (A)
- net 1DIR8: now reaches J1.48
- net 1DIR8: now also U2.5 (QF), D43.2 (A)
- net 1A4STEP: now reaches J1.49
- net 1A4STEP: now also U2.6 (QG), D5.2 (A)
- net 1A8STEP: now reaches J1.50
- net 1A8STEP: now also U2.7 (QH), D44.2 (A)
- net 1A4EN: now reaches J1.51
- net 1A4EN: now also U1.15 (QA), D4.2 (A)
- net 1A8EN: now reaches J1.52
- net 1A8EN: now also U1.1 (QB), D45.2 (A)
- net 1A4MS1: now reaches J1.53
- net 1A4MS1: now also U1.2 (QC), D3.2 (A)
- net 1A8MS1: now reaches J1.54
- net 1A8MS1: now also U1.3 (QD), D46.2 (A)
- net 1A4MS2: now reaches J1.55
- net 1A4MS2: now also U1.4 (QE), D2.2 (A)
- net 1A8MS2: now reaches J1.56
- net 1A8MS2: now also U1.5 (QF), D47.2 (A)
- net 1A4MS3: now reaches J1.57
- net 1A4MS3: now also U1.6 (QG), D1.2 (A)
- net 1A8MS3: now reaches J1.58
- net 1A8MS3: now also U1.7 (QH), D48.2 (A)
- net 4DIR5: now reaches U24.1 (QB)
- net 4DIR5: now also J4.12
- net at U24.14 (SER): now also U23.9 (QH')
- net 4DIR1: now reaches U24.15 (QA)
- net 4DIR1: now also J4.11, D168.2 (A), D192.2 (A)
- net 4A1STEP: now reaches U24.2 (QC)
- net 4A1STEP: now also J4.13, D167.2 (A), D191.2 (A)
- net 4A5STEP: now reaches U24.3 (QD)
- net 4A5STEP: now also J4.14
- net 4A1EN: now reaches U24.4 (QE)
- net 4A1EN: now also J4.15, D166.2 (A), D190.2 (A)
- net 4A5EN: now reaches U24.5 (QF)
- net 4A5EN: now also J4.16
- net 4A1MS1: now reaches U24.6 (QG)
- net 4A1MS1: now also J4.17, D165.2 (A), D189.2 (A)
- net 4A5MS1: now reaches U24.7 (QH)
- net 4A5MS1: now also J4.18
- net at U6.14 (SER): now also U5.9 (QH')
- net at U6.9 (QH'): now also U7.14 (SER)
- net 4A6EN: now reaches U22.1 (QB)
- net 4A6EN: now also J4.28
- net at U22.14 (SER): now also U21.9 (QH')
- net 4A2EN: now reaches U22.15 (QA)
- net 4A2EN: now also J4.27, D160.2 (A), D184.2 (A)
- net 4A2MS1: now reaches U22.2 (QC)
- net 4A2MS1: now also J4.29, D159.2 (A), D183.2 (A)
- net 4A6MS1: now reaches U22.3 (QD)
- net 4A6MS1: now also J4.30
- net 4A2MS2: now reaches U22.4 (QE)
- net 4A2MS2: now also J4.31, D158.2 (A), D182.2 (A)
- net 4A6MS2: now reaches U22.5 (QF)
- net 4A6MS2: now also J4.32
- net 4A2MS3: now reaches U22.6 (QG)
- net 4A2MS3: now also J4.33, D157.2 (A), D181.2 (A)
- net 4A6MS3: now reaches U22.7 (QH)
- net 4A6MS3: now also J4.34
- net at U22.9 (QH'): now also U23.14 (SER)
- net 3A1MS2: now reaches J3.19
- net 3A1MS2: now also U17.15 (QA), D116.2 (A)
- net 3A5MS2: now reaches J3.20
- net 3A5MS2: now also U17.1 (QB), D125.2 (A)
- net 3A1MS3: now reaches J3.21
- net 3A1MS3: now also U17.2 (QC), D115.2 (A)
- net 3A5MS3: now reaches J3.22
- net 3A5MS3: now also U17.3 (QD), D126.2 (A)
- net 3DIR2: now reaches J3.23
- net 3DIR2: now also U17.4 (QE), D114.2 (A)
- net 3DIR6: now reaches J3.24
- net 3DIR6: now also U17.5 (QF), D127.2 (A)
- net 3A2STEP: now reaches J3.25
- net 3A2STEP: now also U17.6 (QG), D113.2 (A)
- net 3A6STEP: now reaches J3.26
- net 3A6STEP: now also U17.7 (QH), D128.2 (A)
- net 3A2EN: now reaches J3.27
- net 3A2EN: now also U16.15 (QA), D112.2 (A)
- net 3A6EN: now reaches J3.28
- net 3A6EN: now also U16.1 (QB), D129.2 (A)
- net 3A2MS1: now reaches J3.29
- net 3A2MS1: now also U16.2 (QC), D111.2 (A)
- net 3A6MS1: now reaches J3.30
- net 3A6MS1: now also U16.3 (QD), D130.2 (A)
- net 3A2MS2: now reaches J3.31
- net 3A2MS2: now also U16.4 (QE), D110.2 (A)
- net 3A6MS2: now reaches J3.32
- net 3A6MS2: now also U16.5 (QF), D131.2 (A)
- net 3A2MS3: now reaches J3.33
- net 3A2MS3: now also U16.6 (QG), D109.2 (A)
- net 3A6MS3: now reaches J3.34
- net 3A6MS3: now also U16.7 (QH), D132.2 (A)
- net 3DIR3: now reaches J3.35
- net 3DIR3: now also U15.15 (QA), D108.2 (A)
- net 3DIR7: now reaches J3.36
- net 3DIR7: now also U15.1 (QB), D133.2 (A)
- net 3A3STEP: now reaches J3.37
- net 3A3STEP: now also U15.2 (QC), D107.2 (A)
- net 3A7STEP: now reaches J3.38
- net 3A7STEP: now also U15.3 (QD), D134.2 (A)
- net 3A3EN: now reaches J3.39
- net 3A3EN: now also U15.4 (QE), D106.2 (A)
- net 3A7EN: now reaches J3.40
- net 3A7EN: now also U15.5 (QF), D135.2 (A)
- net 3A3MS1: now reaches J3.41
- net 3A3MS1: now also U15.6 (QG), D105.2 (A)
- net 3A7MS1: now reaches J3.42
- net 3A7MS1: now also U15.7 (QH), D136.2 (A)
- net 3A3MS2: now reaches J3.43
- net 3A3MS2: now also U14.15 (QA), D104.2 (A)
- net 3A7MS2: now reaches J3.44
- net 3A7MS2: now also U14.1 (QB), D137.2 (A)
- net 3A3MS3: now reaches J3.45
- net 3A3MS3: now also U14.2 (QC), D103.2 (A)
- new net: D91.1 (K), R91.1
- new net: D3.1 (K), R3.1
- new net: D103.1 (K), R103.1
- new net: D8.1 (K), R8.1
- new net: D107.1 (K), R107.1
- new net: D162.1 (K), R162.1
- new net: D164.1 (K), R164.1
- new net: D138.1 (K), R138.1
- new net: D56.1 (K), R56.1
- new net: D125.1 (K), R125.1
- new net: D76.1 (K), R76.1
- new net: D121.1 (K), R121.1
- new net: D166.1 (K), R166.1
- new net: D101.1 (K), R101.1
- new net: D163.1 (K), R163.1
- new net: D173.1 (K), R173.1
- new net: D187.1 (K), R187.1
- new net: D69.1 (K), R69.1
- new net: D94.1 (K), R94.1
- new net: D11.1 (K), R11.1
- new net: D97.1 (K), R97.1
- new net: D180.1 (K), R180.1
- new net: D49.1 (K), R49.1
- new net: D75.1 (K), R75.1
- new net: D18.1 (K), R18.1
- new net: D192.1 (K), R192.1
- new net: D7.1 (K), R7.1
- new net: D73.1 (K), R73.1
- new net: D160.1 (K), R160.1
- new net: D80.1 (K), R80.1
- new net: D77.1 (K), R77.1
- new net: D70.1 (K), R70.1
- new net: D149.1 (K), R149.1
- new net: D141.1 (K), R141.1
- new net: D36.1 (K), R36.1
- new net: D48.1 (K), R48.1
- new net: D53.1 (K), R53.1
- new net: D41.1 (K), R41.1
- new net: D5.1 (K), R5.1
- new net: D106.1 (K), R106.1
- new net: D142.1 (K), R142.1
- new net: D20.1 (K), R20.1
- new net: D111.1 (K), R111.1
- new net: D34.1 (K), R34.1
- new net: D54.1 (K), R54.1
- new net: D133.1 (K), R133.1
- new net: D146.1 (K), R146.1
- new net: D184.1 (K), R184.1
- new net: D86.1 (K), R86.1
- new net: D35.1 (K), R35.1
- new net: D104.1 (K), R104.1
- new net: D15.1 (K), R15.1
- new net: D29.1 (K), R29.1
- new net: D122.1 (K), R122.1
- new net: D47.1 (K), R47.1
- new net: D158.1 (K), R158.1
- new net: D154.1 (K), R154.1
- new net: D96.1 (K), R96.1
- new net: D150.1 (K), R150.1
- new net: D13.1 (K), R13.1
- new net: D55.1 (K), R55.1
- new net: D90.1 (K), R90.1
- new net: D45.1 (K), R45.1
- new net: D64.1 (K), R64.1
- new net: D186.1 (K), R186.1
- new net: D132.1 (K), R132.1
- new net: D144.1 (K), R144.1
- new net: D153.1 (K), R153.1
- new net: D71.1 (K), R71.1
- new net: D38.1 (K), R38.1
- new net: D2.1 (K), R2.1
- new net: D129.1 (K), R129.1
- new net: D119.1 (K), R119.1
- new net: D43.1 (K), R43.1
- new net: D105.1 (K), R105.1
- new net: D102.1 (K), R102.1
- new net: D161.1 (K), R161.1
- new net: D128.1 (K), R128.1
- new net: D155.1 (K), R155.1
- new net: D176.1 (K), R176.1
- new net: D24.1 (K), R24.1
- new net: D179.1 (K), R179.1
- new net: D79.1 (K), R79.1
- new net: D139.1 (K), R139.1
- new net: D57.1 (K), R57.1
- new net: D40.1 (K), R40.1
- new net: D10.1 (K), R10.1
- new net: D131.1 (K), R131.1
- new net: D19.1 (K), R19.1
- new net: D168.1 (K), R168.1
- new net: D16.1 (K), R16.1
- new net: D26.1 (K), R26.1
- new net: D27.1 (K), R27.1
- new net: D67.1 (K), R67.1
- new net: D114.1 (K), R114.1
- new net: D37.1 (K), R37.1
- new net: D98.1 (K), R98.1
- new net: D189.1 (K), R189.1
- new net: D92.1 (K), R92.1
- new net: D152.1 (K), R152.1
- new net: D93.1 (K), R93.1
- new net: D156.1 (K), R156.1
- new net: D140.1 (K), R140.1
- new net: D130.1 (K), R130.1
- new net: D61.1 (K), R61.1
- new net: D82.1 (K), R82.1
- new net: D143.1 (K), R143.1
- new net: D178.1 (K), R178.1
- new net: D181.1 (K), R181.1
- new net: D6.1 (K), R6.1
- new net: D148.1 (K), R148.1
- new net: D136.1 (K), R136.1
- new net: D120.1 (K), R120.1
- new net: D63.1 (K), R63.1
- new net: D108.1 (K), R108.1
- new net: D95.1 (K), R95.1
- new net: D39.1 (K), R39.1
- new net: D46.1 (K), R46.1
- new net: D12.1 (K), R12.1
- new net: D58.1 (K), R58.1
- new net: D99.1 (K), R99.1
- new net: D177.1 (K), R177.1
- new net: D135.1 (K), R135.1
- new net: D172.1 (K), R172.1
- new net: D23.1 (K), R23.1
- new net: D170.1 (K), R170.1
- new net: D74.1 (K), R74.1
- new net: D124.1 (K), R124.1
- new net: D182.1 (K), R182.1
- new net: D25.1 (K), R25.1
- new net: D81.1 (K), R81.1
- new net: D28.1 (K), R28.1
- new net: D68.1 (K), R68.1
- new net: D115.1 (K), R115.1
- new net: D9.1 (K), R9.1
- new net: D171.1 (K), R171.1
- new net: D145.1 (K), R145.1
- new net: D22.1 (K), R22.1
- new net: D88.1 (K), R88.1
- new net: D31.1 (K), R31.1
- new net: D134.1 (K), R134.1
- new net: D4.1 (K), R4.1
- new net: D188.1 (K), R188.1
- new net: D42.1 (K), R42.1
- new net: D51.1 (K), R51.1
- new net: D116.1 (K), R116.1
- new net: D126.1 (K), R126.1
- new net: D87.1 (K), R87.1
- new net: D21.1 (K), R21.1
- new net: D151.1 (K), R151.1
- new net: D123.1 (K), R123.1
- new net: D191.1 (K), R191.1
- new net: D62.1 (K), R62.1
- new net: D50.1 (K), R50.1
- new net: D185.1 (K), R185.1
- new net: D78.1 (K), R78.1
- new net: D113.1 (K), R113.1
- new net: D85.1 (K), R85.1
- new net: D66.1 (K), R66.1
- new net: D112.1 (K), R112.1
- new net: D165.1 (K), R165.1
- new net: D14.1 (K), R14.1
- new net: D159.1 (K), R159.1
- new net: D169.1 (K), R169.1
- new net: D17.1 (K), R17.1
- new net: D183.1 (K), R183.1
- new net: D72.1 (K), R72.1
- new net: D147.1 (K), R147.1
- new net: D52.1 (K), R52.1
- new net: D117.1 (K), R117.1
- new net: D89.1 (K), R89.1
- new net: D137.1 (K), R137.1
- new net: D190.1 (K), R190.1
- new net: D1.1 (K), R1.1
- new net: D60.1 (K), R60.1
- new net: D44.1 (K), R44.1
- new net: D157.1 (K), R157.1
- new net: D175.1 (K), R175.1
- new net: D32.1 (K), R32.1
- new net: D118.1 (K), R118.1
- new net: D84.1 (K), R84.1
- new net: D100.1 (K), R100.1
- new net: D59.1 (K), R59.1
- new net: D174.1 (K), R174.1
- new net: D30.1 (K), R30.1
- new net: D110.1 (K), R110.1
- new net: D65.1 (K), R65.1
- new net: D167.1 (K), R167.1
- new net: D83.1 (K), R83.1
- new net: D33.1 (K), R33.1
- new net: D127.1 (K), R127.1
- new net: D109.1 (K), R109.1
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Other:
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
Commit message: added more connectors
Parts:
- removed D101, D107, D11, D113, D119, D122, D128, D134, D140, D149, D155, D161, D167, D17, D173, D179, D185, D191, D23, D26, D32, D38, D44, D5, D53, D59, D65, D71, D74, D80, D86, D92: LED, symbol Device:LED
- removed R101, R107, R11, R113, R119, R122, R128, R134, R140, R149, R155, R161, R167, R17, R173, R179, R185, R191, R23, R26, R32, R38, R44, R5, R53, R59, R65, R71, R74, R80, R86, R92: R, symbol Device:R
- removed U16, U23, U24, U8: 74HC595, symbol 74xx:74HC595
- added J5: (no value), symbol IPS1-125-01-S-D:IPS1-125-01-S-D
- added J6: (no value), symbol UMPT-06-01-X-RA-WT-P-X:UMPT-06-01-X-RA-WT-P-X
- D1: value (none) -> LED; footprint (none) -> LED_SMD:LED_0603_1608Metric
- D10, D100, D102, D103, D104, D105, D106, D108, D109, D110, D111, D112, D114, D115, D116, D117, D118, D12, D120, D121, D123, D124, D125, D126, D127, D129, D13, D130, D131, D132, D133, D135, D136, D137, D138, D139, D14, D141, D142, D143, D144, D145, D146, D147, D148, D15, D150, D151, D152, D153, D154, D156, D157, D158, D159, D16, D160, D162, D163, D164, D165, D166, D168, D169, D170, D171, D172, D174, D175, D176, D177, D178, D18, D180, D181, D182, D183, D184, D186, D187, D188, D189, D19, D190, D192, D2, D20, D21, D22, D24, D25, D27, D28, D29, D3, D30, D31, D33, D34, D35, D36, D37, D39, D4, D40, D41, D42, D43, D45, D46, D47, D48, D49, D50, D51, D52, D54, D55, D56, D57, D58, D6, D60, D61, D62, D63, D64, D66, D67, D68, D69, D7, D70, D72, D73, D75, D76, D77, D78, D79, D8, D81, D82, D83, D84, D85, D87, D88, D89, D9, D90, D91, D93, D94, D95, D96, D97, D98, D99: footprint (none) -> LED_SMD:LED_0603_1608Metric
- J1, J2, J3, J4: footprint (none) -> LIBRARIES:SAMTEC_MEC2-30-01-X-TH1-NP-WT
- R1: value (none) -> R; footprint (none) -> Resistor_SMD:R_0603_1608Metric
- R10, R100, R102, R103, R104, R105, R106, R108, R109, R110, R111, R112, R114, R115, R116, R117, R118, R12, R120, R121, R123, R124, R125, R126, R127, R129, R13, R130, R131, R132, R133, R135, R136, R137, R138, R139, R14, R141, R142, R143, R144, R145, R146, R147, R148, R15, R150, R151, R152, R153, R154, R156, R157, R158, R159, R16, R160, R162, R163, R164, R165, R166, R168, R169, R170, R171, R172, R174, R175, R176, R177, R178, R18, R180, R181, R182, R183, R184, R186, R187, R188, R189, R19, R190, R192, R2, R20, R21, R22, R24, R25, R27, R28, R29, R3, R30, R31, R33, R34, R35, R36, R37, R39, R4, R40, R41, R42, R43, R45, R46, R47, R48, R49, R50, R51, R52, R54, R55, R56, R57, R58, R6, R60, R61, R62, R63, R64, R66, R67, R68, R69, R7, R70, R72, R73, R75, R76, R77, R78, R79, R8, R81, R82, R83, R84, R85, R87, R88, R89, R9, R90, R91, R93, R94, R95, R96, R97, R98, R99: footprint (none) -> Resistor_SMD:R_0603_1608Metric
- U1, U10, U11, U12, U13, U14, U15, U17, U18, U19, U2, U20, U21, U22, U3, U4, U5, U6, U7, U9: footprint (none) -> Package_SO:TSSOP-16_4.4x5mm_P0.65mm
Connections:
- net +5V: now also J6.01
- net 1A1EN: now also U5.4 (QE); no longer U6.4 (QE)
- net 1A1MS1: now also U5.6 (QG); no longer U6.6 (QG)
- net 1A1MS2: now also U4.4 (QE); no longer U5.15 (QA)
- net 1A1MS3: now also U4.6 (QG); no longer U5.2 (QC)
- net 1A1STEP: now also J5.07; no longer U6.2 (QC)
- net 1A2EN: now also U3.4 (QE); no longer U4.15 (QA)
- net 1A2MS1: now also U3.6 (QG); no longer U4.2 (QC)
- net 1A2MS2: now also U4.15 (QA); no longer U4.4 (QE)
- net 1A2MS3: now also U4.2 (QC); no longer U4.6 (QG)
- net 1A2STEP: now also J5.05; no longer U5.6 (QG)
- net 1A3EN: now also U3.15 (QA); no longer U3.4 (QE)
- net 1A3MS1: now also U3.2 (QC); no longer U3.6 (QG)
- net 1A3STEP: now also J5.03; no longer U3.2 (QC)
- net 1A4STEP: now also J5.01; no longer U2.6 (QG)
- net 1A5EN: now also U5.5 (QF); no longer U6.5 (QF)
- net 1A5MS1: now also U5.7 (QH); no longer U6.7 (QH)
- net 1A5MS2: now also U4.5 (QF); no longer U5.1 (QB)
- net 1A5MS3: now also U4.7 (QH); no longer U5.3 (QD)
- net 1A5STEP: now also J5.08; no longer U6.3 (QD)
- net 1A6EN: now also U3.5 (QF); no longer U4.1 (QB)
- net 1A6MS1: now also U3.7 (QH); no longer U4.3 (QD)
- net 1A6MS2: now also U4.1 (QB); no longer U4.5 (QF)
- net 1A6MS3: now also U4.3 (QD); no longer U4.7 (QH)
- net 1A6STEP: now also J5.06; no longer U5.7 (QH)
- net 1A7EN: now also U3.1 (QB); no longer U3.5 (QF)
- net 1A7MS1: now also U3.3 (QD); no longer U3.7 (QH)
- net 1A7STEP: now also J5.04; no longer U3.3 (QD)
- net 1A8STEP: now also J5.02; no longer U2.7 (QH)
- net 1DIR1: now also U5.2 (QC); no longer U6.15 (QA)
- net 1DIR2: now also U5.15 (QA); no longer U5.4 (QE)
- net 1DIR3: now also U2.6 (QG); no longer U3.15 (QA)
- net 1DIR5: now also U5.3 (QD); no longer U6.1 (QB)
- net 1DIR6: now also U5.1 (QB); no longer U5.5 (QF)
- net 1DIR7: now also U2.7 (QH); no longer U3.1 (QB)
- net 2A1EN: now also U11.4 (QE); no longer U12.4 (QE)
- net 2A1MS1: now also U11.6 (QG); no longer U12.6 (QG)
- net 2A1MS2: now also U10.4 (QE); no longer U11.15 (QA)
- net 2A1MS3: now also U10.6 (QG); no longer U11.2 (QC)
- net 2A1STEP: now also J5.15; no longer U12.2 (QC)
- net 2A2EN: now also U9.4 (QE); no longer U10.15 (QA)
- net 2A2MS1: now also U9.6 (QG); no longer U10.2 (QC)
- net 2A2MS2: now also U10.15 (QA); no longer U10.4 (QE)
- net 2A2MS3: now also U10.2 (QC); no longer U10.6 (QG)
- net 2A2STEP: now also J5.13; no longer U11.6 (QG)
- net 2A3EN: now also U9.15 (QA); no longer U9.4 (QE)
- net 2A3MS1: now also U9.2 (QC); no longer U9.6 (QG)
- net 2A3MS2: now also U7.15 (QA)
- net 2A3MS3: now also U7.2 (QC)
- net 2A3STEP: now also J5.11; no longer U9.2 (QC)
- net 2A4EN: now also U6.15 (QA); no longer U7.15 (QA)
- net 2A4MS1: now also U6.2 (QC); no longer U7.2 (QC)
- net 2A4MS2: now also U6.4 (QE); no longer U7.4 (QE)
- net 2A4MS3: now also U6.6 (QG); no longer U7.6 (QG)
- net 2A4STEP: now also J5.09
- net 2A5EN: now also U11.5 (QF); no longer U12.5 (QF)
- net 2A5MS1: now also U11.7 (QH); no longer U12.7 (QH)
- net 2A5MS2: now also U10.5 (QF); no longer U11.1 (QB)
- net 2A5MS3: now also U10.7 (QH); no longer U11.3 (QD)
- net 2A5STEP: now also J5.16; no longer U12.3 (QD)
- net 2A6EN: now also U9.5 (QF); no longer U10.1 (QB)
- net 2A6MS1: now also U9.7 (QH); no longer U10.3 (QD)
- net 2A6MS2: now also U10.1 (QB); no longer U10.5 (QF)
- net 2A6MS3: now also U10.3 (QD); no longer U10.7 (QH)
- net 2A6STEP: now also J5.14; no longer U11.7 (QH)
- net 2A7EN: now also U9.1 (QB); no longer U9.5 (QF)
- net 2A7MS1: now also U9.3 (QD); no longer U9.7 (QH)
- net 2A7MS2: now also U7.1 (QB)
- net 2A7MS3: now also U7.3 (QD)
- net 2A7STEP: now also J5.12; no longer U9.3 (QD)
- net 2A8EN: now also U6.1 (QB); no longer U7.1 (QB)
- net 2A8MS1: now also U6.3 (QD); no longer U7.3 (QD)
- net 2A8MS2: now also U6.5 (QF); no longer U7.5 (QF)
- net 2A8MS3: now also U6.7 (QH); no longer U7.7 (QH)
- net 2A8STEP: now also J5.10
- net 2DIR1: now also U11.2 (QC); no longer U12.15 (QA)
- net 2DIR2: now also U11.15 (QA); no longer U11.4 (QE)
- net 2DIR3: now also U7.6 (QG); no longer U9.15 (QA)
- net 2DIR4: now also U7.4 (QE)
- net 2DIR5: now also U11.3 (QD); no longer U12.1 (QB)
- net 2DIR6: now also U11.1 (QB); no longer U11.5 (QF)
- net 2DIR7: now also U7.7 (QH); no longer U9.1 (QB)
- net 2DIR8: now also U7.5 (QF)
- net 3A1EN: now also U15.4 (QE); no longer U18.4 (QE)
- net 3A1MS1: now also U15.6 (QG); no longer U18.6 (QG)
- net 3A1MS2: now also U14.4 (QE); no longer U17.15 (QA)
- net 3A1MS3: now also U14.6 (QG); no longer U17.2 (QC)
- net 3A1STEP: no longer U18.2 (QC)
- net 3A2EN: now also U17.15 (QA)
- net 3A2MS1: now also U17.2 (QC)
- net 3A2MS2: now also U17.4 (QE)
- net 3A2MS3: now also U17.6 (QG)
- net 3A2STEP: no longer U17.6 (QG)
- net 3A3EN: now also U14.15 (QA); no longer U15.4 (QE)
- net 3A3MS1: now also U14.2 (QC); no longer U15.6 (QG)
- net 3A3MS2: now also U13.15 (QA); no longer U14.15 (QA)
- net 3A3MS3: now also U13.2 (QC); no longer U14.2 (QC)
- net 3A3STEP: no longer U15.2 (QC)
- net 3A4EN: now also U12.15 (QA); no longer U13.15 (QA)
- net 3A4MS1: now also U12.2 (QC); no longer U13.2 (QC)
- net 3A4MS2: now also U12.4 (QE); no longer U13.4 (QE)
- net 3A4MS3: now also U12.6 (QG); no longer U13.6 (QG)
- net 3A4STEP: no longer U14.6 (QG)
- net 3A5EN: now also U15.5 (QF); no longer U18.5 (QF)
- net 3A5MS1: now also U15.7 (QH); no longer U18.7 (QH)
- net 3A5MS2: now also U14.5 (QF); no longer U17.1 (QB)
- net 3A5MS3: now also U14.7 (QH); no longer U17.3 (QD)
- net 3A5STEP: no longer U18.3 (QD)
- net 3A6EN: now also U17.1 (QB)
- net 3A6MS1: now also U17.3 (QD)
- net 3A6MS2: now also U17.5 (QF)
- net 3A6MS3: now also U17.7 (QH)
- net 3A6STEP: no longer U17.7 (QH)
- net 3A7EN: now also U14.1 (QB); no longer U15.5 (QF)
- net 3A7MS1: now also U14.3 (QD); no longer U15.7 (QH)
- net 3A7MS2: now also U13.1 (QB); no longer U14.1 (QB)
- net 3A7MS3: now also U13.3 (QD); no longer U14.3 (QD)
- net 3A7STEP: no longer U15.3 (QD)
- net 3A8EN: now also U12.1 (QB); no longer U13.1 (QB)
- net 3A8MS1: now also U12.3 (QD); no longer U13.3 (QD)
- net 3A8MS2: now also U12.5 (QF); no longer U13.5 (QF)
- net 3A8MS3: now also U12.7 (QH); no longer U13.7 (QH)
- net 3A8STEP: no longer U14.7 (QH)
- net 3DIR1: now also U15.2 (QC); no longer U18.15 (QA)
- net 3DIR2: now also U15.15 (QA); no longer U17.4 (QE)
- net 3DIR3: now also U13.6 (QG); no longer U15.15 (QA)
- net 3DIR4: now also U13.4 (QE); no longer U14.4 (QE)
- net 3DIR5: now also U15.3 (QD); no longer U18.1 (QB)
- net 3DIR6: now also U15.1 (QB); no longer U17.5 (QF)
- net 3DIR7: now also U13.7 (QH); no longer U15.1 (QB)
- net 3DIR8: now also U13.5 (QF); no longer U14.5 (QF)
- net 4A1EN: now also U22.4 (QE); no longer D190.2 (A)
- net 4A1MS1: now also U22.6 (QG); no longer D189.2 (A)
- net 4A1MS2: now also U21.4 (QE); no longer D188.2 (A)
- net 4A1MS3: now also U21.6 (QG); no longer D187.2 (A)
- net 4A2EN: now also U20.4 (QE); no longer D184.2 (A), U22.15 (QA)
- net 4A2MS1: now also U20.6 (QG); no longer D183.2 (A), U22.2 (QC)
- net 4A2MS2: now also U21.15 (QA); no longer D182.2 (A), U22.4 (QE)
- net 4A2MS3: now also U21.2 (QC); no longer D181.2 (A), U22.6 (QG)
- net 4A3EN: now also U20.15 (QA); no longer D178.2 (A), U21.4 (QE)
- net 4A3MS1: now also U20.2 (QC); no longer D177.2 (A), U21.6 (QG)
- net 4A3MS2: now also U19.15 (QA); no longer D176.2 (A), U20.15 (QA)
- net 4A3MS3: now also U19.2 (QC); no longer D175.2 (A), U20.2 (QC)
- net 4A3STEP: no longer U21.2 (QC)
- net 4A4EN: now also U18.15 (QA); no longer D172.2 (A), U19.15 (QA)
- net 4A4MS1: now also U18.2 (QC); no longer D171.2 (A), U19.2 (QC)
- net 4A4MS2: now also U18.4 (QE); no longer D170.2 (A), U19.4 (QE)
- net 4A4MS3: now also U18.6 (QG); no longer D169.2 (A), U19.6 (QG)
- net 4A4STEP: no longer U20.6 (QG)
- net 4A5EN: now also D174.2 (A), U22.5 (QF)
- net 4A5MS1: now also D175.2 (A), U22.7 (QH)
- net 4A5MS2: now also D176.2 (A), U21.5 (QF)
- net 4A5MS3: now also D177.2 (A), U21.7 (QH)
- net 4A6EN: now also D180.2 (A), U20.5 (QF); no longer U22.1 (QB)
- net 4A6MS1: now also D181.2 (A), U20.7 (QH); no longer U22.3 (QD)
- net 4A6MS2: now also D182.2 (A), U21.1 (QB); no longer U22.5 (QF)
- net 4A6MS3: now also D183.2 (A), U21.3 (QD); no longer U22.7 (QH)
- net 4A7EN: now also D186.2 (A), U20.1 (QB); no longer U21.5 (QF)
- net 4A7MS1: now also D187.2 (A), U20.3 (QD); no longer U21.7 (QH)
- net 4A7MS2: now also D188.2 (A), U19.1 (QB); no longer U20.1 (QB)
- net 4A7MS3: now also D189.2 (A), U19.3 (QD); no longer U20.3 (QD)
- net 4A7STEP: no longer U21.3 (QD)
- net 4A8EN: now also D192.2 (A), U18.1 (QB); no longer U19.1 (QB)
- net 4A8MS1: now also D170.2 (A), U18.3 (QD); no longer U19.3 (QD)
- net 4A8MS2: now also D171.2 (A), U18.5 (QF); no longer U19.5 (QF)
- net 4A8MS3: now also D172.2 (A), U18.7 (QH); no longer U19.7 (QH)
- net 4A8STEP: no longer U20.7 (QH)
- net 4DIR1: now also U22.2 (QC); no longer D192.2 (A)
- net 4DIR2: now also U22.15 (QA); no longer D186.2 (A)
- net 4DIR3: now also U19.6 (QG); no longer D180.2 (A), U21.15 (QA)
- net 4DIR4: now also U19.4 (QE); no longer D174.2 (A), U20.4 (QE)
- net 4DIR5: now also D169.2 (A), U22.3 (QD)
- net 4DIR6: now also D178.2 (A), U22.1 (QB)
- net 4DIR7: now also D184.2 (A), U19.7 (QH); no longer U21.1 (QB)
- net 4DIR8: now also D190.2 (A), U19.5 (QF); no longer U20.5 (QF)
- net GND: now also J6.04, J6.05, J6.06
- net SER2: now also U6.14 (SER); no longer U9.14 (SER)
- net SER3: now also U12.14 (SER); no longer U17.14 (SER)
- net VCC: now also J6.02, J6.03
- net at U17.9 (QH'): no longer U18.14 (SER)
- net at U5.9 (QH'): no longer U6.14 (SER)
- net at U7.9 (QH'): now also U9.14 (SER)
- net at U11.9 (QH'): no longer U12.14 (SER)
- new net SER4: U18.14 (SER)
Other:
- moved on the sheet: D1, D10, D100, D102, D103, D104, D105, D106, D108, D109, D110, D111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

Commit message: progress
Parts:
- J5: value (none) -> IPS1-125-01-S-D; footprint (none) -> LIBRARIES:SAMTEC_IPS1-125-01-S-D
- J6: value (none) -> UMPT-06-01-X-RA-WT-P-X; footprint (none) -> LIBRARIES:SAMTEC_UMPT-06-01-X-RA-WT-P-X
Connections:
- net 3A1STEP: now also J5.23
- net 3A2STEP: now also J5.21
- net 3A3STEP: now also J5.19
- net 3A4STEP: now also J5.17
- net 3A5STEP: now also J5.24
- net 3A6STEP: now also J5.22
- net 3A7STEP: now also J5.20
- net 3A8STEP: now also J5.18
- net 4A1STEP: now also J5.31
- net 4A2STEP: now also J5.29
- net 4A3STEP: now also J5.27
- net 4A4STEP: now also J5.25
- net 4A5STEP: now also J5.32
- net 4A6STEP: now also J5.30
- net 4A7STEP: now also J5.28
- net 4A8STEP: now also J5.26
Changed lines of the file:
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@@
     )
   )
-  (global_label "3A6STEP" (shape input) (at 467.36 86.36 0) (fields_autoplaced)
-    (effects (font (size 1.27 1.27)) (justify left))
-    (property "Intersheet References" "${INTERSHEET_REFS}" (id 0) (at 477.8769 86.2806 0)
-      (effects (font (size 1.27 1.27)) (justify left) hide)
+  (global_label "3A6STEP" (shape input) (at 374.015 97.155 180) (fields_autoplaced)
+    (effects (font (size 1.27 1.27)) (justify right))
+    (property "Intersheet References" "${INTERSHEET_REFS}" (id 0) (at 363.4981 97.2344 0)
+      (effects (font (size 1.27 1.27)) (justify right) hide)
     )
   )
@@
     )
   )
-  (global_label "3A3STEP" (shape input) (at 467.36 78.74 0) (fields_autoplaced)
+  (global_label "3A3STEP" (shape input) (at 399.415 94.615 0) (fields_autoplaced)
     (effects (font (size 1.27 1.27)) (justify left))
-    (property "Intersheet References" "${INTERSHEET_REFS}" (id 0) (at 477.8769 78.6606 0)
+    (property "Intersheet References" "${INTERSHEET_REFS}" (id 0) (at 409.9319 94.5356 0)
       (effects (font (size 1.27 1.27)) (justify left) hide)
     )
@@
     )
   )
-  (global_label "4A6STEP" (shape input) (at 481.33 86.36 0) (fields_autoplaced)
-    (effects (font (size 1.27 1.27)) (justify left))
-    (property "Intersheet References" "${INTERSHEET_REFS}" (id 0) (at 491.8469 86.2806 0)
-      (effects (font (size 1.27 1.27)) (justify left) hide)
+  (global_label "4A6STEP" (shape input) (at 374.015 107.315 180) (fields_autoplaced)
+    (effects (font (size 1.27 1.27)) (justify right))
+    (property "Intersheet References" "${INTERSHEET_REFS}" (id 0) (at 363.4981 107.3944 0)
+      (effects (font (size 1.27 1.27)) (justify right) hide)
     )
   )
@@
     )
   )
-  (global_label "4A2STEP" (shape input) (at 481.33 83.82 0) (fields_autoplaced)
+  (global_label "4A2STEP" (shape input) (at 399.415 107.315 0) (fields_autoplaced)
     (effects (font (size 1.27 1.27)) (justify left))
-    (property "Intersheet References" "${INTERSHEET_REFS}" (id 0) (at 491.8469 83.7406 0)
+    (property "Intersheet References" "${INTERSHEET_REFS}" (id 0) (at 409.9319 107.2356 0)
       (effects (font (size 1.27 1.27)) (justify left) hide)
     )
@@
     )
   )
-  (global_label "4A8STEP" (shape input) (at 481.33 76.2 0) (fields_autoplaced)
-    (effects (font (size 1.27 1.27)) (justify left))
-    (property "Intersheet References" "${INTERSHEET_REFS}" (id 0) (at 491.8469 76.1206 0)
-      (effects (font (size 1.27 1.27)) (justify left) hide)
+  (global_label "4A8STEP" (shape input) (at 374.015 102.235 180) (fields_autoplaced)
+    (effects (font (size 1.27 1.27)) (justify right))
+    (property "Intersheet References" "${INTERSHEET_REFS}" (id 0) (at 363.4981 102.3144 0)
+      (effects (font (size 1.27 1.27)) (justify right) hide)
     )
   )
@@
     )
   )
-  (global_label "4A7STEP" (shape input) (at 481.33 81.28 0) (fields_autoplaced)
-    (effects (font (size 1.27 1.27)) (justify left))
-    (property "Intersheet References" "${INTERSHEET_REFS}" (id 0) (at 491.8469 81.2006 0)
-      (effects (font (size 1.27 1.27)) (justify left) hide)
+  (global_label "4A7STEP" (shape input) (at 374.015 104.775 180) (fields_autoplaced)
+    (effects (font (size 1.27 1.27)) (justify right))
+    (property "Intersheet References" "${INTERSHEET_REFS}" (id 0) (at 363.4981 104.8544 0)
+      (effects (font (size 1.27 1.27)) (justify right) hide)
     )
   )
@@
     )
   )
-  (global_label "3A7STEP" (shape input) (at 467.36 81.28 0) (fields_autoplaced)
-    (effects (font (size 1.27 1.27)) (justify left))
-    (property "Intersheet References" "${INTERSHEET_REFS}" (id 0) (at 477.8769 81.2006 0)
-      (effects (font (size 1.27 1.27)) (justify left) hide)
+  (global_label "3A7STEP" (shape input) (at 374.015 94.615 180) (fields_autoplaced)
+    (effects (font (size 1.27 1.27)) (justify right))
+    (property "Intersheet References" "${INTERSHEET_REFS}" (id 0) (at 363.4981 94.6944 0)
+      (effects (font (size 1.27 1.27)) (justify right) hide)
     )
   )
@@
     )
   )
-  (global_label "4A1STEP" (shape input) (at 481.33 88.9 0) (fields_autoplaced)
+  (global_label "4A1STEP" (shape input) (at 399.415 109.855 0) (fields_autoplaced)
     (effects (font (size 1.27 1.27)) (justify left))
-    (property "Intersheet References" "${INTERSHEET_REFS}" (id 0) (at 491.8469 88.8206 0)
+    (property "Intersheet References" "${INTERSHEET_REFS}" (id 0) (at 409.9319 109.7756 0)
       (effects (font (size 1.27 1.27)) (justify left) hide)
     )
@@
     )
   )
-  (global_label "4A5STEP" (shape input) (at 481.33 91.44 0) (fields_autoplaced)
-    (effects (font (size 1.27 1.27)) (justify left))
-    (property "Intersheet References" "${INTERSHEET_REFS}" (id 0) (at 491.8469 91.3606 0)
-      (effects (font (size 1.27 1.27)) (justify left) hide)
+  (global_label "4A5STEP" (shape input) (at 374.015 109.855 180) (fields_autoplaced)
+    (effects (font (size 1.27 1.27)) (justify right))
+    (property "Intersheet References" "${INTERSHEET_REFS}" (id 0) (at 363.4981 109.9344 0)
+      (effects (font (size 1.27 1.27)) (justify right) hide)
     )
   )
@@
     )
   )
-  (global_label "3A4STEP" (shape input) (at 467.36 73.66 0) (fields_autoplaced)
+  (global_label "3A4STEP" (shape input) (at 399.415 92.075 0) (fields_autoplaced)
     (effects (font (size 1.27 1.27)) (justify left))
-    (property "Intersheet References" "${INTERSHEET_REFS}" (id 0) (at 477.8769 73.5806 0)
+    (property "Intersheet References" "${INTERSHEET_REFS}" (id 0) (at 409.9319 91.9956 0)
       (effects (font (size 1.27 1.27)) (justify left) hide)
     )
@@
     )
   )
-  (global_label "3A1STEP" (shape input) (at 467.36 88.9 0) (fields_autoplaced)
+  (global_label "3A1STEP" (shape input) (at 399.415 99.695 0) (fields_autoplaced)
     (effects (font (size 1.27 1.27)) (justify left))
-    (property "Intersheet References" "${INTERSHEET_REFS}" (id 0) (at 477.8769 88.8206 0)
+    (property "Intersheet References" "${INTERSHEET_REFS}" (id 0) (at 409.9319 99.6156 0)
       (effects (font (size 1.27 1.27)) (justify left) hide)
     )
@@
     )
   )
-  (global_label "3A2STEP" (shape input) (at 467.36 83.82 0) (fields_autoplaced)
+  (global_label "3A2STEP" (shape input) (at 399.415 97.155 0) (fields_autoplaced)
     (effects (font (size 1.27 1.27)) (justify left))
-    (property "Intersheet References" "${INTERSHEET_REFS}" (id 0) (at 477.8769 83.7406 0)
+    (property "Intersheet References" "${INTERSHEET_REFS}" (id 0) (at 409.9319 97.0756 0)
       (effects (font (size 1.27 1.27)) (justify left) hide)
     )
@@
     )
   )
-  (global_label "3A5STEP" (shape input) (at 467.36 91.44 0) (fields_autoplaced)
-    (effects (font (size 1.27 1.27)) (justify left))
-    (property "Intersheet References" "${INTERSHEET_REFS}" (id 0) (at 477.8769 91.3606 0)
-      (effects (font (size 1.27 1.27)) (justify left) hide)
+  (global_label "3A5STEP" (shape input) (at 374.015 99.695 180) (fields_autoplaced)
+    (effects (font (size 1.27 1.27)) (justify right))
+    (property "Intersheet References" "${INTERSHEET_REFS}" (id 0) (at 363.4981 99.7744 0)
+      (effects (font (size 1.27 1.27)) (justify right) hide)
     )
   )
@@
     )
   )
-  (global_label "4A3STEP" (shape input) (at 481.33 78.74 0) (fields_autoplaced)
+  (global_label "4A3STEP" (shape input) (at 399.415 104.775 0) (fields_autoplaced)
     (effects (font (size 1.27 1.27)) (justify left))
-    (property "Intersheet References" "${INTERSHEET_REFS}" (id 0) (at 491.8469 78.6606 0)
+    (property "Intersheet References" "${INTERSHEET_REFS}" (id 0) (at 409.9319 104.6956 0)
       (effects (font (size 1.27 1.27)) (justify left) hide)
     )
@@
     )
   )
-  (global_label "4A4STEP" (shape input) (at 481.33 73.66 0) (fields_autoplaced)
+  (global_label "4A4STEP" (shape input) (at 399.415 102.235 0) (fields_autoplaced)
     (effects (font (size 1.27 1.27)) (justify left))
-    (property "Intersheet References" "${INTERSHEET_REFS}" (id 0) (at 491.8469 73.5806 0)
+    (property "Intersheet References" "${INTERSHEET_REFS}" (id 0) (at 409.9319 102.1556 0)
       (effects (font (size 1.27 1.27)) (justify left) hide)
     )
@@
     )
   )
-  (global_label "3A8STEP" (shape input) (at 467.36 76.2 0) (fields_autoplaced)
-    (effects (font (size 1.27 1.27)) (justify left))
-    (property "Intersheet References" "${INTERSHEET_REFS}" (id 0) (at 477.8769 76.1206 0)
-      (effects (font (size 1.27 1.27)) (justify left) hide)
+  (global_label "3A8STEP" (shape input) (at 374.015 92.075 180) (fields_autoplaced)
+    (effects (font (size 1.27 1.27)) (justify right))
+    (property "Intersheet References" "${INTERSHEET_REFS}" (id 0) (at 363.4981 92.1544 0)
+      (effects (font (size 1.27 1.27)) (justify right) hide)
     )
   )
@@
       (effects (font (size 1.27 1.27)) (justify left))
     )
-    (property "Value" "" (id 1) (at 387.985 179.07 0)
+    (property "Value" "UMPT-06-01-X-RA-WT-P-X" (id 1) (at 387.985 179.07 0)
       (effects (font (size 1.27 1.27)) (justify left))
     )
-    (property "Footprint" "" (id 2) (at 394.335 167.005 0)
+    (property "Footprint" "LIBRARIES:SAMTEC_UMPT-06-01-X-RA-WT-P-X" (id 2) (at 394.335 167.005 0)
       (effects (font (size 1.27 1.27)) (justify left bottom) hide)
     )
@@
     (in_bom yes) (on_board yes) (fields_autoplaced)
     (property "Reference" "J5" (id 0) (at 386.715 65.5152 0))
-    (property "Value" "" (id 1) (at 386.715 68.0521 0))
-    (property "Footprint" "" (id 2) (at 386.715 102.235 0)
+    (property "Value" "IPS1-125-01-S-D" (id 1) (at 386.715 68.0521 0))
+    (property "Footprint" "LIBRARIES:SAMTEC_IPS1-125-01-S-D" (id 2) (at 386.715 102.235 0)
       (effects (font (size 1.27 1.27)) (justify left bottom) hide)
     )
