File: PCB/32-STEPPER-DRIVER-BOARD/32-STEPPER-DRIVER-BOARD.kicad_sch (KiCad schematic)
At the start: 346 parts, among them J1 MEC2-30-01-X-TH1-NP-WT, J2 MEC2-30-01-X-TH1-NP-WT, J3 MEC2-30-01-X-TH1-NP-WT, J4 MEC2-30-01-X-TH1-NP-WT, J5 IPS1-125-01-S-D, J6 UMPT-06-01-X-RA-WT-P-X, U1 74HC595, U10 74HC595, U11 74HC595, U12 74HC595, U13 74HC595, U14 74HC595, U15 74HC595, U17 74HC595, U18 74HC595, U19 74HC595, U2 74HC595, U20 74HC595, U21 74HC595, U22 74HC595, U3 74HC595, U4 74HC595, U5 74HC595, U6 74HC595, U7 74HC595, U9 74HC595

Commit message: re-routing bottom layer
Parts:
- renumbered U17 to U16, U18 to U17, U19 to U18, U20 to U19, U21 to U20, U22 to U21
Connections:
- net 1A1EN: now also U5.2 (QC); no longer U5.4 (QE)
- net 1A1MS1: now also U5.4 (QE); no longer U5.6 (QG)
- net 1A1MS2: now also U5.6 (QG); no longer U4.4 (QE)
- net 1A1MS3: now also U4.15 (QA); no longer U4.6 (QG)
- net 1A2EN: now also U4.4 (QE); no longer U3.4 (QE)
- net 1A2MS1: now also U4.6 (QG); no longer U3.6 (QG)
- net 1A2MS2: now also U3.15 (QA); no longer U4.15 (QA)
- net 1A2MS3: now also U3.2 (QC); no longer U4.2 (QC)
- net 1A3EN: now also U3.6 (QG); no longer U3.15 (QA)
- net 1A3MS1: now also U2.15 (QA); no longer U3.2 (QC)
- net 1A3MS2: now also U2.2 (QC); no longer U2.15 (QA)
- net 1A3MS3: now also U2.4 (QE); no longer U2.2 (QC)
- net 1A5EN: now also U5.3 (QD); no longer U5.5 (QF)
- net 1A5MS1: now also U5.5 (QF); no longer U5.7 (QH)
- net 1A5MS2: now also U5.7 (QH); no longer U4.5 (QF)
- net 1A5MS3: now also U4.1 (QB); no longer U4.7 (QH)
- net 1A6EN: now also U4.5 (QF); no longer U3.5 (QF)
- net 1A6MS1: now also U4.7 (QH); no longer U3.7 (QH)
- net 1A6MS2: now also U3.1 (QB); no longer U4.1 (QB)
- net 1A6MS3: now also U3.3 (QD); no longer U4.3 (QD)
- net 1A7EN: now also U3.7 (QH); no longer U3.1 (QB)
- net 1A7MS1: now also U2.1 (QB); no longer U3.3 (QD)
- net 1A7MS2: now also U2.3 (QD); no longer U2.1 (QB)
- net 1A7MS3: now also U2.5 (QF); no longer U2.3 (QD)
- net 1DIR1: now also U5.15 (QA); no longer U5.2 (QC)
- net 1DIR2: now also U4.2 (QC); no longer U5.15 (QA)
- net 1DIR3: now also U3.4 (QE); no longer U2.6 (QG)
- net 1DIR4: now also U2.6 (QG); no longer U2.4 (QE)
- net 1DIR5: now also U5.1 (QB); no longer U5.3 (QD)
- net 1DIR6: now also U4.3 (QD); no longer U5.1 (QB)
- net 1DIR7: now also U3.5 (QF); no longer U2.7 (QH)
- net 1DIR8: now also U2.7 (QH); no longer U2.5 (QF)
- net 2A1EN: now also U11.2 (QC); no longer U11.4 (QE)
- net 2A1MS1: now also U11.4 (QE); no longer U11.6 (QG)
- net 2A1MS2: now also U11.6 (QG); no longer U10.4 (QE)
- net 2A1MS3: now also U10.15 (QA); no longer U10.6 (QG)
- net 2A2EN: now also U10.4 (QE); no longer U9.4 (QE)
- net 2A2MS1: now also U10.6 (QG); no longer U9.6 (QG)
- net 2A2MS2: now also U9.15 (QA); no longer U10.15 (QA)
- net 2A2MS3: now also U9.2 (QC); no longer U10.2 (QC)
- net 2A3EN: now also U9.6 (QG); no longer U9.15 (QA)
- net 2A3MS1: now also U7.15 (QA); no longer U9.2 (QC)
- net 2A3MS2: now also U7.2 (QC); no longer U7.15 (QA)
- net 2A3MS3: now also U7.4 (QE); no longer U7.2 (QC)
- net 2A5EN: now also U11.3 (QD); no longer U11.5 (QF)
- net 2A5MS1: now also U11.5 (QF); no longer U11.7 (QH)
- net 2A5MS2: now also U11.7 (QH); no longer U10.5 (QF)
- net 2A5MS3: now also U10.1 (QB); no longer U10.7 (QH)
- net 2A6EN: now also U10.5 (QF); no longer U9.5 (QF)
- net 2A6MS1: now also U10.7 (QH); no longer U9.7 (QH)
- net 2A6MS2: now also U9.1 (QB); no longer U10.1 (QB)
- net 2A6MS3: now also U9.3 (QD); no longer U10.3 (QD)
- net 2A7EN: now also U9.7 (QH); no longer U9.1 (QB)
- net 2A7MS1: now also U7.1 (QB); no longer U9.3 (QD)
- net 2A7MS2: now also U7.3 (QD); no longer U7.1 (QB)
- net 2A7MS3: now also U7.5 (QF); no longer U7.3 (QD)
- net 2DIR1: now also U11.15 (QA); no longer U11.2 (QC)
- net 2DIR2: now also U10.2 (QC); no longer U11.15 (QA)
- net 2DIR3: now also U9.4 (QE); no longer U7.6 (QG)
- net 2DIR4: now also U7.6 (QG); no longer U7.4 (QE)
- net 2DIR5: now also U11.1 (QB); no longer U11.3 (QD)
- net 2DIR6: now also U10.3 (QD); no longer U11.1 (QB)
- net 2DIR7: now also U9.5 (QF); no longer U7.7 (QH)
- net 2DIR8: now also U7.7 (QH); no longer U7.5 (QF)
- net 3A2EN: now also U16.2 (QC); no longer U16.15 (QA)
- net 3A2MS1: now also U16.4 (QE); no longer U16.2 (QC)
- net 3A2MS2: now also U16.6 (QG); no longer U16.4 (QE)
- net 3A2MS3: now also U15.15 (QA); no longer U16.6 (QG)
- net 3A6EN: now also U16.3 (QD); no longer U16.1 (QB)
- net 3A6MS1: now also U16.5 (QF); no longer U16.3 (QD)
- net 3A6MS2: now also U16.7 (QH); no longer U16.5 (QF)
- net 3A6MS3: now also U15.1 (QB); no longer U16.7 (QH)
- net 3DIR2: now also U16.15 (QA); no longer U15.15 (QA)
- net 3DIR6: now also U16.1 (QB); no longer U15.1 (QB)

Commit message: cleanup before DRC Errors
Parts:
- added JP1: (no value), symbol Jumper:SolderJumper_2_Open
- added JP2: SolderJumper_2_Open, symbol Jumper:SolderJumper_2_Open
Connections:
- net 3A1EN: now also U16.2 (QC); no longer U15.4 (QE)
- net 3A1MS1: now also U16.4 (QE); no longer U15.6 (QG)
- net 3A1MS2: now also U16.6 (QG); no longer U14.4 (QE)
- net 3A1MS3: now also U15.15 (QA); no longer U14.6 (QG)
- net 3A2EN: now also U15.4 (QE); no longer U16.2 (QC)
- net 3A2MS1: now also U15.6 (QG); no longer U16.4 (QE)
- net 3A2MS2: now also U14.15 (QA); no longer U16.6 (QG)
- net 3A2MS3: now also U14.2 (QC); no longer U15.15 (QA)
- net 3A3EN: now also U14.6 (QG); no longer U14.15 (QA)
- net 3A3MS1: now also U13.15 (QA); no longer U14.2 (QC)
- net 3A3MS2: now also U13.2 (QC); no longer U13.15 (QA)
- net 3A3MS3: now also U13.4 (QE); no longer U13.2 (QC)
- net 3A5EN: now also U16.3 (QD); no longer U15.5 (QF)
- net 3A5MS1: now also U16.5 (QF); no longer U15.7 (QH)
- net 3A5MS2: now also U16.7 (QH); no longer U14.5 (QF)
- net 3A5MS3: now also U15.1 (QB); no longer U14.7 (QH)
- net 3A6EN: now also U15.5 (QF); no longer U16.3 (QD)
- net 3A6MS1: now also U15.7 (QH); no longer U16.5 (QF)
- net 3A6MS2: now also U14.1 (QB); no longer U16.7 (QH)
- net 3A6MS3: now also U14.3 (QD); no longer U15.1 (QB)
- net 3A7EN: now also U14.7 (QH); no longer U14.1 (QB)
- net 3A7MS1: now also U13.1 (QB); no longer U14.3 (QD)
- net 3A7MS2: now also U13.3 (QD); no longer U13.1 (QB)
- net 3A7MS3: now also U13.5 (QF); no longer U13.3 (QD)
- net 3DIR1: now also U16.15 (QA); no longer U15.2 (QC)
- net 3DIR2: now also U15.2 (QC); no longer U16.15 (QA)
- net 3DIR3: now also U14.4 (QE); no longer U13.6 (QG)
- net 3DIR4: now also U13.6 (QG); no longer U13.4 (QE)
- net 3DIR5: now also U16.1 (QB); no longer U15.3 (QD)
- net 3DIR6: now also U15.3 (QD); no longer U16.1 (QB)
- net 3DIR7: now also U14.5 (QF); no longer U13.7 (QH)
- net 3DIR8: now also U13.7 (QH); no longer U13.5 (QF)
- net 4A1EN: now also U21.2 (QC); no longer U21.4 (QE)
- net 4A1MS1: now also U21.4 (QE); no longer U21.6 (QG)
- net 4A1MS2: now also U21.6 (QG); no longer U20.4 (QE)
- net 4A1MS3: now also U20.15 (QA); no longer U20.6 (QG)
- net 4A2EN: now also U20.4 (QE); no longer U19.4 (QE)
- net 4A2MS1: now also U20.6 (QG); no longer U19.6 (QG)
- net 4A2MS2: now also U19.15 (QA); no longer U20.15 (QA)
- net 4A2MS3: now also U19.2 (QC); no longer U20.2 (QC)
- net 4A3EN: now also U19.6 (QG); no longer U19.15 (QA)
- net 4A3MS1: now also U18.15 (QA); no longer U19.2 (QC)
- net 4A3MS2: now also U18.2 (QC); no longer U18.15 (QA)
- net 4A3MS3: now also U18.4 (QE); no longer U18.2 (QC)
- net 4A5EN: now also U21.3 (QD); no longer U21.5 (QF)
- net 4A5MS1: now also U21.5 (QF); no longer U21.7 (QH)
- net 4A5MS2: now also U21.7 (QH); no longer U20.5 (QF)
- net 4A5MS3: now also U20.1 (QB); no longer U20.7 (QH)
- net 4A6EN: now also U20.5 (QF); no longer U19.5 (QF)
- net 4A6MS1: now also U20.7 (QH); no longer U19.7 (QH)
- net 4A6MS2: now also U19.1 (QB); no longer U20.1 (QB)
- net 4A6MS3: now also U19.3 (QD); no longer U20.3 (QD)
- net 4A7EN: now also U19.7 (QH); no longer U19.1 (QB)
- net 4A7MS1: now also U18.1 (QB); no longer U19.3 (QD)
- net 4A7MS2: now also U18.3 (QD); no longer U18.1 (QB)
- net 4A7MS3: now also U18.5 (QF); no longer U18.3 (QD)
- net 4DIR1: now also U21.15 (QA); no longer U21.2 (QC)
- net 4DIR2: now also U20.2 (QC); no longer U21.15 (QA)
- net 4DIR3: now also U19.4 (QE); no longer U18.6 (QG)
- net 4DIR4: now also U18.6 (QG); no longer U18.4 (QE)
- net 4DIR5: now also U21.1 (QB); no longer U21.3 (QD)
- net 4DIR6: now also U20.3 (QD); no longer U21.1 (QB)
- net 4DIR7: now also U19.5 (QF); no longer U18.7 (QH)
- net 4DIR8: now also U18.7 (QH); no longer U18.5 (QF)
- net GND: now also J6.02, JP1.2 (B), JP2.2 (B); no longer J6.05, R1.2, R10.2, R100.2, R102.2, R103.2, R104.2, R105.2, R106.2, R108.2, R109.2, R110.2, R111.2, R112.2, R114.2, R115.2, R116.2, R117.2, R118.2, R12.2, R120.2, R121.2, R123.2, R124.2, R125.2, R126.2, R127.2, R129.2, R13.2, R130.2, R131.2, R132.2, R133.2, R135.2, R136.2, R137.2, R138.2, R139.2, R14.2, R141.2, R142.2, R143.2, R144.2, R145.2, R146.2, R147.2, R148.2, R15.2, R150.2, R151.2, R152.2, R153.2, R154.2, R156.2, R157.2, R158.2, R159.2, R16.2, R160.2, R162.2, R163.2, R164.2, R165.2, R166.2, R168.2, R169.2, R170.2, R171.2, R172.2, R174.2, R175.2, R176.2, R177.2, R178.2, R18.2, R180.2, R181.2, R182.2, R183.2, R184.2, R186.2, R187.2, R188.2, R189.2, R19.2, R190.2, R192.2, R2.2, R20.2, R21.2, R22.2, R24.2, R25.2, R27.2, R28.2, R29.2, R3.2, R30.2, R31.2, R33.2, R34.2, R35.2, R36.2, R37.2, R39.2, R4.2, R40.2, R41.2, R42.2, R43.2, R45.2, R46.2, R47.2, R48.2, R49.2, R50.2, R51.2, R52.2, R54.2, R55.2, R56.2, R57.2, R58.2, R6.2, R60.2, R61.2, R62.2, R63.2, R64.2, R66.2, R67.2, R68.2, R69.2, R7.2, R70.2, R72.2, R73.2, R75.2, R76.2, R77.2, R78.2, R79.2, R8.2, R81.2, R82.2, R83.2, R84.2, R85.2, R87.2, R88.2, R89.2, R9.2, R90.2, R91.2, R93.2, R94.2, R95.2, R96.2, R97.2, R98.2, R99.2
- net RCLK: now also J5.38
- net SER1: now also J5.33
- net SER2: now also J5.40
- net SER3: now also J5.42
- net SER4: now also J5.44
- net VCC: now also J6.05; no longer J6.02
- net ~{OE}: now also J5.37
- net ~{SRCLR}: now also J5.36
- net at U16.14 (SER): now also U15.9 (QH')
- net SRCLK1: now reaches J5.34
- net SRCLK1: now also U1.11 (SRCLK), U2.11 (SRCLK), U3.11 (SRCLK), U4.11 (SRCLK), U5.11 (SRCLK)
- net SRCLK2: now reaches J5.35
- net SRCLK2: now also U10.11 (SRCLK), U11.11 (SRCLK), U6.11 (SRCLK), U7.11 (SRCLK), U9.11 (SRCLK)
- net SRCLK3: now reaches J5.39
- net SRCLK3: now also U12.11 (SRCLK), U13.11 (SRCLK), U14.11 (SRCLK), U15.11 (SRCLK), U16.11 (SRCLK)
- net SRCLK4: now reaches J5.41
- net SRCLK4: now also U17.11 (SRCLK), U18.11 (SRCLK), U19.11 (SRCLK), U20.11 (SRCLK), U21.11 (SRCLK)
- removed net SRCLK: U1.11 (SRCLK), U10.11 (SRCLK), U11.11 (SRCLK), U12.11 (SRCLK), U13.11 (SRCLK), U14.11 (SRCLK), U15.11 (SRCLK), U16.11 (SRCLK), U17.11 (SRCLK), U18.11 (SRCLK), U19.11 (SRCLK), U2.11 (SRCLK), U20.11 (SRCLK), U21.11 (SRCLK), U3.11 (SRCLK), U4.11 (SRCLK), U5.11 (SRCLK), U6.11 (SRCLK), U7.11 (SRCLK), U9.11 (SRCLK)
- new net GND1: JP1.1 (A), R1.2, R10.2, R12.2, R13.2, R14.2, R15.2, R16.2, R18.2, R19.2, R2.2, R20.2, R21.2, R22.2, R24.2, R25.2, R27.2, R28.2, R29.2, R3.2, R30.2, R31.2, R33.2, R34.2, R35.2, R36.2, R37.2, R39.2, R4.2, R40.2, R41.2, R42.2, R43.2, R45.2, R46.2, R47.2, R48.2, R49.2, R50.2, R51.2, R52.2, R54.2, R55.2, R56.2, R57.2, R58.2, R6.2, R60.2, R61.2, R62.2, R63.2, R64.2, R66.2, R67.2, R68.2, R69.2, R7.2, R70.2, R72.2, R73.2, R75.2, R76.2, R77.2, R78.2, R79.2, R8.2, R81.2, R82.2, R83.2, R84.2, R85.2, R87.2, R88.2, R89.2, R9.2, R90.2, R91.2, R93.2, R94.2, R95.2, R96.2
- new net GND2: JP2.1 (A), R100.2, R102.2, R103.2, R104.2, R105.2, R106.2, R108.2, R109.2, R110.2, R111.2, R112.2, R114.2, R115.2, R116.2, R117.2, R118.2, R120.2, R121.2, R123.2, R124.2, R125.2, R126.2, R127.2, R129.2, R130.2, R131.2, R132.2, R133.2, R135.2, R136.2, R137.2, R138.2, R139.2, R141.2, R142.2, R143.2, R144.2, R145.2, R146.2, R147.2, R148.2, R150.2, R151.2, R152.2, R153.2, R154.2, R156.2, R157.2, R158.2, R159.2, R160.2, R162.2, R163.2, R164.2, R165.2, R166.2, R168.2, R169.2, R170.2, R171.2, R172.2, R174.2, R175.2, R176.2, R177.2, R178.2, R180.2, R181.2, R182.2, R183.2, R184.2, R186.2, R187.2, R188.2, R189.2, R190.2, R192.2, R97.2, R98.2, R99.2

Commit message: final adjustments
Parts:
- added J10, J7, J8, J9: Screw_Terminal_01x01, MountingHole:MountingHole_2.2mm_M2_Pad, symbol Connector:Screw_Terminal_01x01
- JP1: value (none) -> SolderJumper_2_Open; footprint (none) -> Jumper:SolderJumper-2_P1.3mm_Open_RoundedPad1.0x1.5mm
- JP2: footprint (none) -> Jumper:SolderJumper-2_P1.3mm_Open_RoundedPad1.0x1.5mm
Connections:
- net +5V: now also J5.45, J5.46
- net GND: now also J5.47, J5.48, J5.49, J5.50, J10.1 (Pin_1), J7.1 (Pin_1), J8.1 (Pin_1), J9.1 (Pin_1)
- net VCC: now also J5.43

Commit message: Create BOM for 32-Board
Parts:
- D1, D10, D100, D102, D103, D104, D105, D106, D108, D109, D110, D111, D112, D114, D115, D116, D117, D118, D12, D120, D121, D123, D124, D125, D126, D127, D129, D13, D130, D131, D132, D133, D135, D136, D137, D138, D139, D14, D141, D142, D143, D144, D145, D146, D147, D148, D15, D150, D151, D152, D153, D154, D156, D157, D158, D159, D16, D160, D162, D163, D164, D165, D166, D168, D169, D170, D171, D172, D174, D175, D176, D177, D178, D18, D180, D181, D182, D183, D184, D186, D187, D188, D189, D19, D190, D192, D2, D20, D21, D22, D24, D25, D27, D28, D29, D3, D30, D31, D33, D34, D35, D36, D37, D39, D4, D40, D41, D42, D43, D45, D46, D47, D48, D49, D50, D51, D52, D54, D55, D56, D57, D58, D6, D60, D61, D62, D63, D64, D66, D67, D68, D69, D7, D70, D72, D73, D75, D76, D77, D78, D79, D8, D81, D82, D83, D84, D85, D87, D88, D89, D9, D90, D91, D93, D94, D95, D96, D97, D98, D99: manf# (none) -> B1931NB--20C007614U1930
- J1, J2, J3, J4: manf# (none) -> MEC2-30-01-L-TH1-NP-WT
- J5: manf# (none) -> IPT1-125-01-S-D
- J6: manf# (none) -> UMPT-06-01-L-RA-WT-P-TR
- R1, R10, R100, R102, R103, R104, R105, R106, R108, R109, R110, R111, R112, R114, R115, R116, R117, R118, R12, R120, R121, R123, R124, R125, R126, R127, R129, R13, R130, R131, R132, R133, R135, R136, R137, R138, R139, R14, R141, R142, R143, R144, R145, R146, R147, R148, R15, R150, R151, R152, R153, R154, R156, R157, R158, R159, R16, R160, R162, R163, R164, R165, R166, R168, R169, R170, R171, R172, R174, R175, R176, R177, R178, R18, R180, R181, R182, R183, R184, R186, R187, R188, R189, R19, R190, R192, R2, R20, R21, R22, R24, R25, R27, R28, R29, R3, R30, R31, R33, R34, R35, R36, R37, R39, R4, R40, R41, R42, R43, R45, R46, R47, R48, R49, R50, R51, R52, R54, R55, R56, R57, R58, R6, R60, R61, R62, R63, R64, R66, R67, R68, R69, R7, R70, R72, R73, R75, R76, R77, R78, R79, R8, R81, R82, R83, R84, R85, R87, R88, R89, R9, R90, R91, R93, R94, R95, R96, R97, R98, R99: manf# (none) -> RC0603FR-071KL
- U1, U10, U11, U12, U13, U14, U15, U16, U17, U18, U19, U2, U20, U21, U3, U4, U5, U6, U7, U9: manf# (none) -> MC74HC595ADTG
