File: PCB/64-STEPPER-CONTROLLER/64-STEPPER-CONTROLLER.kicad_sch (KiCad schematic)
At the start: 19 parts, among them J1 IPS1-125-01-S-D, J10 UMPT-02-01-X-RA-WT-P-X, J11 Conn_01x03, J12 Conn_01x03, J13 Conn_01x09, J14 Screw_Terminal_01x01, J15 Screw_Terminal_01x01, J2 IPS1-125-01-S-D, J3 Conn_01x03, J4 Conn_01x03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

Commit message: final changes to 64-pcb and testing renders
Connections:
- net LED1: now also J12.2 (Pin_2); no longer J3.2 (Pin_2)
- net LED5: now also J3.2 (Pin_2); no longer J7.2 (Pin_2)
- net LED9: now also J7.2 (Pin_2); no longer J12.2 (Pin_2)
