File: PCB/2-STEPPER-BREAKOUT/2-STEPPER-BREAKOUT.kicad_sch (KiCad schematic)
At the start: 3 parts, among them J1 Conn_01x04_Female, J2 Conn_01x04_Female, J3 Conn_01x08

Commit message: Create BOM for 32-Board
Changed lines of the file:
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@@
   (symbol (lib_id "Connector:Conn_01x04_Female") (at 151.765 68.58 0) (mirror y) (unit 1)
     (in_bom yes) (on_board yes)
-    (property "Reference" "J1" (id 0) (at 152.4 78.74 0))
+    (property "Reference" "J1" (id 0) (at 148.59 69.85 0))
     (property "Value" "Conn_01x04_Female" (id 1) (at 151.765 86.36 0))
     (property "Footprint" "Connector_PinSocket_2.54mm:PinSocket_1x04_P2.54mm_Horizontal" (id 2) (at 151.765 68.58 0)
@@
   (symbol (lib_id "Connector:Conn_01x04_Female") (at 151.765 78.74 0) (mirror y) (unit 1)
     (in_bom yes) (on_board yes)
-    (property "Reference" "J2" (id 0) (at 152.4 76.2 0))
+    (property "Reference" "J2" (id 0) (at 148.59 78.74 0))
     (property "Value" "Conn_01x04_Female" (id 1) (at 151.765 62.23 0))
     (property "Footprint" "Connector_PinSocket_2.54mm:PinSocket_1x04_P2.54mm_Horizontal" (id 2) (at 151.765 78.74 0)
