File: PCB/PIANO_LEDS/PIANO_LEDS.kicad_pcb (KiCad board)
At the start: 2 copper layers, 56 x 26 mm, 30 parts, among them J1 Conn_01x03, J2 Conn_01x05_Pin, J3 Conn_01x05_Pin, J4 Conn_01x05_Pin, J5 Conn_01x05_Pin

Commit message: Design complete
Parts:
- removed C12: 100n, Capacitor_SMD:C_0603_1608Metric
- removed C14: 10u, Capacitor_SMD:C_1206_3216Metric
- removed J1: Conn_01x03, libraries:3-PIN TERMINAL
- J2, J3, J4, J5: value Conn_01x05_Pin -> Conn_01x03_Pin
- moved J2 8.02 mm to (51.5, 92.0)
- moved J3 8.02 mm to (106.5, 92.0)
- moved J4 8.02 mm to (106.5, 92.0)
- moved J5 8.02 mm to (51.5, 92.0)
- moved C11 2.00 mm to (103.0, 84.0)
- moved C4 2.00 mm to (71.0, 84.0)
- moved C7 2.00 mm to (87.0, 84.0)
- moved C9 2.00 mm to (95.0, 84.0)
- moved C1 1.58 mm to (58.5, 93.5)
- moved C3 1.58 mm to (66.5, 93.5)
- moved C6 1.58 mm to (82.5, 93.5)
- moved C8 1.58 mm to (90.5, 93.5)
- moved C5 0.90 mm to (74.5, 93.5)
- moved C10 0.71 mm to (98.5, 93.5)
- moved C2 0.25 mm to (63.0, 84.0)
Connections:
- J2 pad 1: GND -> +5V
- J2 pad 2: +5V -> DIN
- J2 pad 3: DIN -> GND
- J3 pad 1: GND -> +5V
- J3 pad 2: +5V -> DOUT
- J3 pad 3: DOUT -> GND
- J4 pad 1: GND -> +5V
- J4 pad 2: +5V -> DOUT
- J4 pad 3: DOUT -> GND
- J5 pad 1: GND -> +5V
- J5 pad 2: +5V -> DIN
- J5 pad 3: DIN -> GND
Routing:
- net +5V: track 9.77 -> 176.2 mm
- net Net-(D10-DOUT): track 0.00 -> 16.0 mm
- net Net-(D8-DOUT): track 0.00 -> 16.0 mm
- net GND: track 0.00 -> 11.5 mm, vias 0 -> 16
- net DOUT: track 0.00 -> 10.5 mm
- net Net-(D11-DOUT): track 0.00 -> 4.39 mm
- net Net-(D10-DIN): track 0.00 -> 4.39 mm
- net DIN: track 7.65 -> 3.40 mm
- net Net-(D1-DOUT): track 15.3 -> 16.0 mm
- net Net-(D3-DOUT): track 15.3 -> 16.0 mm
- added copper zone on B.Cu, net GND
- added copper zone on F.Cu, net GND
Other:
- board size 56 x 26 mm -> 56 x 20 mm
- board text added: "Elliot Eickholtz"
- board text added: "PIANO_LEDS"
- board text added: "REV A"
