File: PCB/PIANO_LEDS/PIANO_LEDS.kicad_sch (KiCad schematic)
At the start: 30 parts, among them J1 Conn_01x03, J2 Conn_01x05_Pin, J3 Conn_01x05_Pin, J4 Conn_01x05_Pin, J5 Conn_01x05_Pin

Commit message: Design complete
Parts:
- removed C12: 100n, Capacitor_SMD:C_0603_1608Metric, symbol Device:C_Small
- removed C14: 10u, Capacitor_SMD:C_1206_3216Metric, symbol Device:C_Small
- removed J1: Conn_01x03, libraries:3-PIN TERMINAL, symbol Connector_Generic:Conn_01x03
- removed J2, J3, J4, J5: Conn_01x05_Pin, libraries:3-PIN_SOLDER_EDGE, symbol Connector:Conn_01x05_Pin
- added J2, J3, J4, J5: Conn_01x03_Pin, libraries:3-PIN_SOLDER_EDGE, symbol Connector:Conn_01x03_Pin
Connections:
- net +5V: now also J2.1 (Pin_1), J3.1 (Pin_1), J4.1 (Pin_1), J5.1 (Pin_1)
- net DIN: now also J2.2 (Pin_2), J5.2 (Pin_2)
- net DOUT: now also J3.2 (Pin_2), J4.2 (Pin_2)
- net GND: now also J2.3 (Pin_3), J3.3 (Pin_3), J4.3 (Pin_3), J5.3 (Pin_3)
